Commit message: 添加手臂相机的moveit，但是没有rviz和gazebo，没有建立连接。出错原因不知道，我的电脑rqt  出错，不给启动

File: rokae/src/rokae_desk/urdf/robot_tool.xacro (robot description, xacro)
@@ -292,9 +292,9 @@
     <type>transmission_interface/SimpleTransmission</type>
     <joint name="xmate_joint_7">
-<hardwareInterface>hardware_interface/PositionJointInterface</hardwareInterface>
+    <hardwareInterface>hardware_interface/PositionJointInterface</hardwareInterface>
     </joint>
     <actuator name="motor7">
-<hardwareInterface>hardware_interface/PositionJointInterface</hardwareInterface>
-      <mechanicalReduction>1</mechanicalReduction>
+    <hardwareInterface>hardware_interface/PositionJointInterface</hardwareInterface>
+    <mechanicalReduction>1</mechanicalReduction>
     </actuator>
   </transmission>

File: rokae/src/rokae_desk/urdf/robot_tool_complex copy.xacro (robot description, xacro)
@@ -32,13 +32,2 @@
   </joint>
 </robot>
-  <!-- <joint name="location_camera_joint" type="fixed">
-    <origin xyz="0 0.15 1.75" rpy="0 3.14 1.57"/>
-    <parent link="rokae_link7"/>
-    <child link="world_base"/>
-  </joint> -->
-  <!-- <sensor_d435 parent="rokae_link7" name="camera_location">
-    <origin xyz="0  -0.1 0" rpy="0 -1.57 1.57"/>
-  </sensor_d435>
-  <sensor_d435 parent="table" name="camera_global">
-    <origin xyz="0.20 0 1.75" rpy="0 1.57 0"/>
-  </sensor_d435> -->
