Commit message: 机器人颜色修改】

File: rokae/src/rokae_desk/urdf/robot.xacro (robot description, xacro)
@@ -52,5 +52,5 @@
   </transmission>
   <gazebo reference="${nameofManipulator}_base">
-     <material>Gazebo/Black</material>
+     <material>Gazebo/GreyTransparent</material>
   </gazebo>
 <!--link 1-->
@@ -93,5 +93,5 @@
   </transmission>
   <gazebo reference="${nameofManipulator}_link1">
-     <material>Gazebo/Black</material>
+     <material>Gazebo/GreyTransparent</material>
   </gazebo>
 <!--link 2-->
@@ -134,5 +134,5 @@
   </transmission>
   <gazebo reference="${nameofManipulator}_link2">
-     <material>Gazebo/Black</material>
+     <material>Gazebo/GreyTransparent</material>
   </gazebo>
 <!--${nameofManipulator}_link 3-->
@@ -177,5 +177,5 @@
   </transmission>
   <gazebo reference="${nameofManipulator}_link3">
-     <material>Gazebo/Black</material>
+     <material>Gazebo/GreyTransparent</material>
   </gazebo>
 <!--link 4-->
@@ -218,5 +218,5 @@
   </transmission>
   <gazebo reference="${nameofManipulator}_link4">
-     <material>Gazebo/Black</material>
+     <material>Gazebo/GreyTransparent</material>
   </gazebo>
 <!--link 5-->
@@ -259,5 +259,5 @@
   </transmission>
   <gazebo reference="${nameofManipulator}_link5">
-     <material>Gazebo/Black</material>
+     <material>Gazebo/GreyTransparent</material>
   </gazebo>
 <!--link 6-->
@@ -300,5 +300,5 @@
   </transmission>
   <gazebo reference="${nameofManipulator}_link6">
-     <material>Gazebo/Black</material>
+     <material>Gazebo/GreyTransparent</material>
   </gazebo>
 <!--link 7-->
@@ -343,5 +343,5 @@
   </transmission> -->
   <gazebo reference="${nameofManipulator}_link7">
-     <material>Gazebo/Black</material>
+     <material>Gazebo/GreyTransparent</material>
   </gazebo>
 <!-- ros_control plugin -->
