Commit message: 同上

File: rokae/src/rokae_desk/urdf/robot_tool_complex.xacro (robot description, xacro)
@@ -5,5 +5,6 @@
   <xacro:include filename="$(find rokae_desk)/urdf/battery_pack.urdf" />
   <xacro:include filename="$(find rokae_desk)/urdf/camera_taotong.urdf" />
-  <xacro:include filename="$(find realsense2_description)/urdf/tool_d435_camera.urdf.xacro"   />
+  <xacro:include filename="$(find realsense2_description)/urdf/test_d435_camera.urdf.xacro"   />
+  <xacro:include filename="$(find realsense2_description)/urdf/gloal_d435_camera.urdf.xacro"   />
   <joint name="table_ur5_joint" type="fixed">
     <origin xyz="-0.55 0 0.12" rpy="0 0 0" />
@@ -21,8 +22,13 @@
     <child link="tool_base_link"/>
   </joint>
-  <joint name="location_camera_joint" type="fixed">
-    <origin xyz="0 0.15 1.75" rpy="0 3.14 1.57"/>
-    <parent link="tool_base_link"/>
-    <child link="camera_base_link"/>
+  <joint name="arm_camera_joint" type="fixed">
+    <origin xyz="0 -0.1 0" rpy="0 -1.57 1.57"/>
+    <parent link="rokae_link7"/>
+    <child link="world_base"/>
+  </joint>
+  <joint name="scene_camera_joint" type="fixed">
+    <origin xyz="0 0 1.75" rpy="0 1.57 1.57"/>
+    <parent link="table"/>
+    <child link="gloal_world_base"/>
   </joint>
 </robot>

Commit message: adjust for capture good picture
1. add gazebo tag to set the battery pack color.
2. adjust the position of rs in arm

File: rokae/src/rokae_desk/urdf/robot_tool_complex.xacro (robot description, xacro)
@@ -23,5 +23,5 @@
   </joint>
   <joint name="arm_camera_joint" type="fixed">
-    <origin xyz="0 -0.1 0" rpy="0 -1.57 1.57"/>
+    <origin xyz="0 -0.05 0" rpy="0 -1.57 1.57"/>
     <parent link="rokae_link7"/>
     <child link="world_base"/>

Commit message: 桌子围栏

File: rokae/src/rokae_desk/urdf/robot_tool_complex.xacro (robot description, xacro)
@@ -7,4 +7,10 @@
   <xacro:include filename="$(find realsense2_description)/urdf/test_d435_camera.urdf.xacro"   />
   <xacro:include filename="$(find realsense2_description)/urdf/gloal_d435_camera.urdf.xacro"   />
+  <xacro:include filename="$(find battery_pack_describe)/urdf/weilan.urdf" />
+  <joint name="weilan_joint" type="fixed">
+    <origin xyz="0 0 0.05" rpy="0 0 0" />
+    <parent link="table"/>
+    <child link="weilan"/>
+  </joint>
   <joint name="table_ur5_joint" type="fixed">
     <origin xyz="-0.55 0 0.12" rpy="0 0 0" />

Commit message: adjust and add code for concept demo

File: rokae/src/rokae_desk/urdf/robot_tool_complex.xacro (robot description, xacro)
@@ -29,5 +29,5 @@
   </joint>
   <joint name="arm_camera_joint" type="fixed">
-    <origin xyz="0 -0.05 0" rpy="0 -1.57 1.57"/>
+    <origin xyz="0 -0.04 0.05" rpy="0 -1.57 1.57"/>
     <parent link="rokae_link7"/>
     <child link="world_base"/>

Commit message: camera  image   x,y,w,h.

File: rokae/src/rokae_desk/urdf/robot_tool_complex.xacro (robot description, xacro)
@@ -34,5 +34,5 @@
   </joint>
   <joint name="scene_camera_joint" type="fixed">
-    <origin xyz="0 0 1.55" rpy="0 1.57 1.57"/>
+    <origin xyz="0 0 1.50" rpy="0 1.57 1.57"/>
     <parent link="table"/>
     <child link="gloal_world_base"/>

Commit message: adjust the camera position for better image quality. add some test image modified the code of bolt detection for trial.

File: rokae/src/rokae_desk/urdf/robot_tool_complex.xacro (robot description, xacro)
@@ -29,5 +29,5 @@
   </joint>
   <joint name="arm_camera_joint" type="fixed">
-    <origin xyz="0 -0.04 0.05" rpy="0 -1.57 1.57"/>
+    <origin xyz="0 -0.02 0.20" rpy="0 -1.57 1.57"/>
     <parent link="rokae_link7"/>
     <child link="world_base"/>

Commit message: adjust camera position according to the size change of taotong.

File: rokae/src/rokae_desk/urdf/robot_tool_complex.xacro (robot description, xacro)
@@ -29,5 +29,5 @@
   </joint>
   <joint name="arm_camera_joint" type="fixed">
-    <origin xyz="0 -0.02 0.20" rpy="0 -1.57 1.57"/>
+    <origin xyz="0 -0.02 0.10" rpy="0 -1.57 1.57"/>
     <parent link="rokae_link7"/>
     <child link="world_base"/>
