Commit message: Link gazebo with moveit for the world arm_camera sucessfully
1. urdf is inconsistent between gazebo and moveit
2. add no collision checking in srdf
3. keep the namespace consistent
4. don't import libgazeros 2 times, esspecially with inconsistent namespace.

File: rokae/src/rokae_desk/urdf/camera_taotong.urdf (robot description, URDF)
Before this commit: robot camera_taotong, 2 links, 1 joints
Links:
- removed link tool_Link
- added link tool_link, mass 0.0282087806682537; collision mesh filename=package://rokae_desk/meshes/tool_Link.stl; visual mesh filename=package://rokae_desk/meshes/tool_Link.stl
Joints:
- joint tool_taotong: child tool_Link -> tool_link

File: rokae/src/rokae_desk/urdf/robot_tool_complex.xacro (robot description, xacro)
@@ -5,5 +5,5 @@
   <xacro:include filename="$(find rokae_desk)/urdf/battery_pack.urdf" />
   <xacro:include filename="$(find rokae_desk)/urdf/camera_taotong.urdf" />
-  <xacro:include filename="$(find realsense2_description)/urdf/test_d435_camera.urdf.xacro"   />
+  <xacro:include filename="$(find realsense2_description)/urdf/tool_d435_camera.urdf.xacro"   />
   <joint name="table_ur5_joint" type="fixed">
     <origin xyz="-0.55 0 0.12" rpy="0 0 0" />
@@ -23,6 +23,6 @@
   <joint name="location_camera_joint" type="fixed">
     <origin xyz="0 0.15 1.75" rpy="0 3.14 1.57"/>
-    <parent link="rokae_link7"/>
-    <child link="world_base"/>
+    <parent link="tool_base_link"/>
+    <child link="camera_base_link"/>
   </joint>
 </robot>

Commit message: 套筒的碰撞盒

File: rokae/src/rokae_desk/urdf/camera_taotong.urdf (robot description, URDF)
Before this commit: robot rokea, 2 links, 1 joints
Links:
- link tool_link: geometry collision cylinder length=0.04 radius=0.02; visual mesh filename=package://rokae_desk/meshes/tool_Link.stl scale=1.25 1.25 1.25

File: rokae/src/rokae_desk/urdf/camera_taotong.xacro (robot description, xacro)
@@ -23,4 +23,5 @@
     <collision>
       <geometry>
+        <cylinder length="0.04" radius="0.2"/>
         <mesh          filename="package://rokae_desk/meshes/tool_base_link.stl" />
       </geometry>
@@ -68,4 +69,5 @@
     <collision>
       <geometry>
+        <cylinder length="0.3" radius="0.02"/>
         <mesh          filename="package://rokae_desk/meshes/tool_Link.stl" />
       </geometry>
