Commit message: 修改了电池包

File: rokae/src/rokae_desk/urdf/camera_taotong.xacro (robot description, xacro)
@@ -45,5 +45,5 @@
   </transmission>
   <gazebo reference="tool_base_link">
-     <material>Gazebo/Green</material>
+     <material>Gazebo/Red</material>
   </gazebo>
 <!-- tool_Link -->
@@ -51,5 +51,5 @@
     <visual>
       <geometry>
-        <mesh          filename="package://rokae_desk/meshes/tool_Link.stl"  scale="1.25 1.25 1.25"/>
+        <mesh          filename="package://rokae_desk/meshes/tool_Link.stl"  scale="1.3 1.3 1.3"/>
       </geometry>
 	    <origin rpy="0 0 0" xyz="0 0 0"/>
@@ -64,6 +64,5 @@
         iyy="0.000106"
         iyz="-1.185"
-        izz="6.544" />
-      <origin        xyz="5.20417042793042E-18 3.79470760369927E-19 -0.0550139882029437"        rpy="0 0 0" />
+        izz="6.544" />      <origin        xyz="5.20417042793042E-18 3.79470760369927E-19 -0.0550139882029437"        rpy="0 0 0" />
     </inertial>
     <collision>
@@ -75,5 +74,6 @@
   </link>
   <gazebo reference="tool_Link">
-     <material>Gazebo/BlackTransparent</material>
+     <!-- <material>Gazebo/BlackTransparent</material> -->
+     <material>Gazebo/Red</material>
   </gazebo>
 <!-- ros_control plugin

Commit message: 套筒也是，不好加碰撞盒

File: rokae/src/rokae_desk/urdf/camera_taotong.xacro (robot description, xacro)
@@ -69,5 +69,5 @@
     <collision>
       <geometry>
-        <cylinder length="0.3" radius="0.02"/>
+        <!-- <cylinder length="0.02" radius="0.02"/> -->
         <mesh          filename="package://rokae_desk/meshes/tool_Link.stl" />
       </geometry>
