Commit message: fix the realsense camera to right position
add joint to connect baselink frame to the world frame

File: rokae/src/realsense-ros-development/realsense2_description/urdf/test_d435_camera.urdf.xacro (robot description, xacro)
@@ -2,5 +2,10 @@
 <robot name="realsense2_camera" xmlns:xacro="http://ros.org/wiki/xacro">
   <xacro:include filename="$(find realsense2_description)/urdf/_d435.urdf.xacro" />
+  <link name="world" />
   <link name="base_link" />
+    <joint name="world_to_base_link" type="fixed">
+        <parent link="world"/>
+        <child link="base_link"/>
+    </joint>
   <xacro:sensor_d435 name="camera" topics_ns="camera" parent="base_link" publish_pointcloud="true">
     <origin xyz="0.25 0 1.75" rpy="0 1.57 0"/>

Commit message: 相机添加

File: rokae/src/realsense-ros-development/realsense2_description/urdf/test_d435_camera.urdf.xacro (robot description, xacro)
@@ -2,8 +2,8 @@
 <robot name="realsense2_camera" xmlns:xacro="http://ros.org/wiki/xacro">
   <xacro:include filename="$(find realsense2_description)/urdf/_d435.urdf.xacro" />
-  <link name="world" />
+  <link name="world_base" />
   <link name="base_link" />
     <joint name="world_to_base_link" type="fixed">
-        <parent link="world"/>
+        <parent link="world_base"/>
         <child link="base_link"/>
     </joint>

File: rokae/src/rokae_desk/urdf/robot.xacro (robot description, xacro)
@@ -323,5 +323,5 @@
     </collision>
   </link>
-  <joint name="xmate_joint_8" type="revolute">
+  <!-- <joint name="xmate_joint_8" type="revolute">
     <parent link="${nameofManipulator}_link7"/>
     <child link="${nameofManipulator}_link8"/>
@@ -339,5 +339,5 @@
       <mechanicalReduction>1</mechanicalReduction>
     </actuator>
-  </transmission>
+  </transmission> -->
   <gazebo reference="${nameofManipulator}_link7">
      <material>Gazebo/Block</material>

File: rokae/src/rokae_desk/urdf/robot_tool_complex.xacro (robot description, xacro)
@@ -2,8 +2,11 @@
 <robot name="rokae" xmlns:xacro="http://www.ros.org/wiki/xacro">
   <!--Used to attach gripper to the UR5 robot -->
-  <xacro:include filename="$(find rokae_desk)/urdf/rokae_robot.xacro" />
+  <xacro:include filename="$(find rokae_desk)/urdf/robot.xacro" />
   <!-- <xacro:include filename="$(find rokae_desk)/urdf/taotong_hed.xacro" /> -->
   <xacro:include filename="$(find cai_env)/urdf/table.urdf.xacro" />
   <xacro:include filename="$(find rokae_desk)/urdf/battery_pack.urdf" />
+  <xacro:include filename="$(find rokae_desk)/urdf/camera_taotong.urdf" />
+  <xacro:include filename="$(find realsense2_description)/urdf/test_d435_camera.urdf.xacro" />
+<!-- 桌子 -->
   <joint name="table_ur5_joint" type="fixed">
     <origin xyz="-0.55 0 0.12" rpy="0 0 0" />
@@ -11,4 +14,5 @@
     <child link="rokae_base"/>
   </joint>
+<!-- 电池包 -->
   <joint name="battery_pack_joint" type="fixed">
     <origin xyz="0 0 0.12" rpy="0 0 3.14" />
@@ -16,9 +20,16 @@
     <child link="battery_pack_link"/>
   </joint>
-  <!-- <joint name="taotong_joint" type="continuous">
-    <origin xyz="0 0 0" rpy="0 0 0" />
+<!-- 拆解工具 -->
+  <joint name="hold_tool_joint" type="fixed">
+    <origin xyz="0 0 0" rpy="0 3.14 0.15" />
     <parent link="rokae_link7"/>
-    <child link="taotong_link8"/>
+    <child link="tool_base_link"/>
   </joint>
-   -->
+<!-- 手臂相机 -->
+  <joint name="location_camera_joint" type="fixed">
+    <origin xyz="0  0   0" rpy="0 0 0"/>
+    <parent link="zhijia_Link"/>
+    <child link="world_base"/>
+  </joint>
+    <!-- <origin xyz="-0.25 0 -1.75" rpy="0 0 0"/> -->
 </robot>

Commit message: 手臂相机

File: rokae/src/realsense-ros-development/realsense2_description/urdf/test_d435_camera.urdf.xacro (robot description, xacro)
@@ -9,5 +9,6 @@
     </joint>
   <xacro:sensor_d435 name="camera" topics_ns="camera" parent="base_link" publish_pointcloud="true">
-    <origin xyz="0.25 0 1.75" rpy="0 1.57 0"/>
+    <!-- <origin xyz="0.25 0 1.75" rpy="0 1.57 0"/> -->
+    <origin xyz="0 0 0" rpy="0 0 0"/>
   </xacro:sensor_d435>
 </robot>

File: rokae/src/rokae_desk/urdf/camera_taotong.urdf (robot description, URDF)
Before this commit: robot camera_taotong, 3 links, 2 joints
Links:
- removed link zhijia_Link
Joints:
- removed joint zhijia_joint

File: rokae/src/rokae_desk/urdf/robot_tool_complex.xacro (robot description, xacro)
@@ -7,5 +7,6 @@
   <xacro:include filename="$(find rokae_desk)/urdf/battery_pack.urdf" />
   <xacro:include filename="$(find rokae_desk)/urdf/camera_taotong.urdf" />
-  <xacro:include filename="$(find realsense2_description)/urdf/test_d435_camera.urdf.xacro" />
+  <xacro:include filename="$(find realsense2_description)/urdf/test_d435_camera.urdf.xacro"   />
+  <!-- <xacro:include filename="$(find realsense2_description)/urdf/test_d435_camera.urdf.xacro"    name="global"  /> -->
 <!-- 桌子 -->
   <joint name="table_ur5_joint" type="fixed">
@@ -28,8 +29,9 @@
 <!-- 手臂相机 -->
   <joint name="location_camera_joint" type="fixed">
-    <origin xyz="0  0   0" rpy="0 0 0"/>
-    <parent link="zhijia_Link"/>
+    <origin xyz="0.1 0 0" rpy="0 1.57 0"/>
+    <parent link="tool_base_link"/>
     <child link="world_base"/>
   </joint>
+    <!-- <origin xyz="-0.40 0 -1.75" rpy="0 0 0"/> -->
     <!-- <origin xyz="-0.25 0 -1.75" rpy="0 0 0"/> -->
 </robot>

Commit message: 添加手臂相机

File: rokae/src/realsense-ros-development/realsense2_description/urdf/test_d435_camera.urdf.xacro (robot description, xacro)
@@ -9,6 +9,6 @@
     </joint>
   <xacro:sensor_d435 name="camera" topics_ns="camera" parent="base_link" publish_pointcloud="true">
-    <!-- <origin xyz="0.25 0 1.75" rpy="0 1.57 0"/> -->
-    <origin xyz="0 0 0" rpy="0 0 0"/>
+    <origin xyz="0.25 0 1.75" rpy="0 1.57 0"/>
+    <!-- <origin xyz="0 0 0" rpy="0 0 0"/> -->
   </xacro:sensor_d435>
 </robot>

File: rokae/src/realsense-ros-development/realsense2_description/urdf/test_d435_multiple_cameras.urdf.xacro (robot description, xacro)
@@ -2,9 +2,10 @@
 <robot name="realsense2_camera" xmlns:xacro="http://ros.org/wiki/xacro">
   <xacro:include filename="$(find realsense2_description)/urdf/_d435.urdf.xacro" />
-  <link name="base_link" />
-  <sensor_d435 parent="base_link" name="camera1">
+  <link name="arm_link" />
+  <link name="gloal_link" />
+  <sensor_d435 parent="arm_link" name="camera1">
     <origin xyz="0 0 1" rpy="0 1.57 0"/>
   </sensor_d435>
-  <sensor_d435 parent="base_link" name="camera2">
+  <sensor_d435 parent="gloal_link" name="camera2">
     <origin xyz="-0.1 0 0" rpy="0 0 3.1456"/>
   </sensor_d435>

File: rokae/src/rokae_desk/urdf/robot.xacro (robot description, xacro)
@@ -44,8 +44,8 @@
     <type>transmission_interface/SimpleTransmission</type>
     <joint name="xmate_joint_1">
-      <hardwareInterface>hardware_interface/PositionJointInterface</hardwareInterface>
+<hardwareInterface>hardware_interface/PositionJointInterface</hardwareInterface>
     </joint>
     <actuator name="motor1">
-      <hardwareInterface>hardware_interface/PositionJointInterface</hardwareInterface>
+<hardwareInterface>hardware_interface/PositionJointInterface</hardwareInterface>
       <mechanicalReduction>1</mechanicalReduction>
     </actuator>
@@ -85,8 +85,8 @@
      <type>transmission_interface/SimpleTransmission</type>
     <joint name="xmate_joint_2">
-      <hardwareInterface>hardware_interface/PositionJointInterface</hardwareInterface>
+<hardwareInterface>hardware_interface/PositionJointInterface</hardwareInterface>
     </joint>
     <actuator name="motor2">
-      <hardwareInterface>hardware_interface/PositionJointInterface</hardwareInterface>
+<hardwareInterface>hardware_interface/PositionJointInterface</hardwareInterface>
       <mechanicalReduction>1</mechanicalReduction>
     </actuator>
@@ -121,13 +121,13 @@
   <limit effort="300" lower="-3.0527" upper="3.0527" velocity="10"/>
     <axis xyz="0 0 1"/>
-    <origin rpy="0 0 0" xyz="0 0 0.23743878"/>_desk
+    <origin rpy="0 0 0" xyz="0 0 0.23743878"/>
   </joint>
    <transmission name="tran3">
     <type>transmission_interface/SimpleTransmission</type>
     <joint name="xmate_joint_3">
-      <hardwareInterface>hardware_interface/PositionJointInterface</hardwareInterface>
+<hardwareInterface>hardware_interface/PositionJointInterface</hardwareInterface>
     </joint>
     <actuator name="motor3">
-      <hardwareInterface>hardware_interface/PositionJointInterface</hardwareInterface>
+<hardwareInterface>hardware_interface/PositionJointInterface</hardwareInterface>
       <mechanicalReduction>1</mechanicalReduction>
     </actuator>
@@ -169,8 +169,8 @@
     <type>transmission_interface/SimpleTransmission</type>
     <joint name="xmate_joint_4">
-      <hardwareInterface>hardware_interface/PositionJointInterface</hardwareInterface>
+<hardwareInterface>hardware_interface/PositionJointInterface</hardwareInterface>
     </joint>
     <actuator name="motor4">
-      <hardwareInterface>hardware_interface/PositionJointInterface</hardwareInterface>
+<hardwareInterface>hardware_interface/PositionJointInterface</hardwareInterface>
       <mechanicalReduction>1</mechanicalReduction>
     </actuator>
@@ -210,8 +210,8 @@
     <type>transmission_interface/SimpleTransmission</type>
     <joint name="xmate_joint_5">
-      <hardwareInterface>hardware_interface/PositionJointInterface</hardwareInterface>
+<hardwareInterface>hardware_interface/PositionJointInterface</hardwareInterface>
     </joint>
     <actuator name="motor5">
-      <hardwareInterface>hardware_interface/PositionJointInterface</hardwareInterface>
+<hardwareInterface>hardware_interface/PositionJointInterface</hardwareInterface>
       <mechanicalReduction>1</mechanicalReduction>
     </actuator>
@@ -251,8 +251,8 @@
     <type>transmission_interface/SimpleTransmission</type>
     <joint name="xmate_joint_6">
-      <hardwareInterface>hardware_interface/PositionJointInterface</hardwareInterface>
+<hardwareInterface>hardware_interface/PositionJointInterface</hardwareInterface>
     </joint>
     <actuator name="motor6">
-      <hardwareInterface>hardware_interface/PositionJointInterface</hardwareInterface>
+<hardwareInterface>hardware_interface/PositionJointInterface</hardwareInterface>
       <mechanicalReduction>1</mechanicalReduction>
     </actuator>
@@ -292,8 +292,8 @@
     <type>transmission_interface/SimpleTransmission</type>
     <joint name="xmate_joint_7">
-      <hardwareInterface>hardware_interface/PositionJointInterface</hardwareInterface>
+<hardwareInterface>hardware_interface/PositionJointInterface</hardwareInterface>
     </joint>
     <actuator name="motor7">
-      <hardwareInterface>hardware_interface/PositionJointInterface</hardwareInterface>
+<hardwareInterface>hardware_interface/PositionJointInterface</hardwareInterface>
       <mechanicalReduction>1</mechanicalReduction>
     </actuator>
@@ -308,5 +308,5 @@
         <mesh filename="package://${nameofManipulator}_desk/meshes/visual/${nameofManipulator}_link7.stl" scale="0.001 0.001 0.001"/>
       </geometry>
-	<origin rpy="0 0 0" xyz="0 0 0"/>
+	    <origin rpy="0 0 0" xyz="0 0 0"/>
       <material name="white"/>
     </visual>
@@ -320,21 +320,23 @@
         <mesh filename="package://${nameofManipulator}_desk/meshes/collision/${nameofManipulator}_link7.stl" scale="0.001 0.001 0.001"/>
       </geometry>
-	<origin rpy="0 0 0" xyz="0 0 0"/>
-    </collision>
-  </link>
-  <!-- <joint name="xmate_joint_8" type="revolute">
+	    <origin rpy="0 0 0" xyz="0 0 0"/>
+    </collision>
+  </link>
+<!--
+    <joint name="xmate_joint_8" type="revolute">
     <parent link="${nameofManipulator}_link7"/>
-    <child link="${nameofManipulator}_link8"/>
-   <limit effort="300" lower="-6.283" upper="6.283" velocity="10"/>
+    <child link="taotong_link8"/>
+      <limit effort="300" lower="-6.283" upper="6.283" velocity="10"/>
     <axis xyz="0 0 1"/>
     <origin rpy="0.0 0.0 0.0" xyz="0 0 0.25090877" />
-  </joint>
-  <transmission name="tran8">
+    </joint>
+   -->
+  <!-- <transmission name="tran8">
     <type>transmission_interface/SimpleTransmission</type>
     <joint name="xmate_joint_8">
-      <hardwareInterface>hardware_interface/PositionJointInterface</hardwareInterface>
+<hardwareInterface>hardware_interface/PositionJointInterface</hardwareInterface>
     </joint>
     <actuator name="motor8">
-      <hardwareInterface>hardware_interface/PositionJointInterface</hardwareInterface>
+<hardwareInterface>hardware_interface/PositionJointInterface</hardwareInterface>
       <mechanicalReduction>1</mechanicalReduction>
     </actuator>

File: rokae/src/rokae_desk/urdf/robot_tool_complex.xacro (robot description, xacro)
@@ -1,13 +1,9 @@
 <?xml version="1.0"?>
 <robot name="rokae" xmlns:xacro="http://www.ros.org/wiki/xacro">
-  <!--Used to attach gripper to the UR5 robot -->
   <xacro:include filename="$(find rokae_desk)/urdf/robot.xacro" />
-  <!-- <xacro:include filename="$(find rokae_desk)/urdf/taotong_hed.xacro" /> -->
   <xacro:include filename="$(find cai_env)/urdf/table.urdf.xacro" />
   <xacro:include filename="$(find rokae_desk)/urdf/battery_pack.urdf" />
   <xacro:include filename="$(find rokae_desk)/urdf/camera_taotong.urdf" />
   <xacro:include filename="$(find realsense2_description)/urdf/test_d435_camera.urdf.xacro"   />
-  <!-- <xacro:include filename="$(find realsense2_description)/urdf/test_d435_camera.urdf.xacro"    name="global"  /> -->
-<!-- 桌子 -->
   <joint name="table_ur5_joint" type="fixed">
     <origin xyz="-0.55 0 0.12" rpy="0 0 0" />
@@ -15,5 +11,4 @@
     <child link="rokae_base"/>
   </joint>
-<!-- 电池包 -->
   <joint name="battery_pack_joint" type="fixed">
     <origin xyz="0 0 0.12" rpy="0 0 3.14" />
@@ -21,17 +16,13 @@
     <child link="battery_pack_link"/>
   </joint>
-<!-- 拆解工具 -->
-  <joint name="hold_tool_joint" type="fixed">
-    <origin xyz="0 0 0" rpy="0 3.14 0.15" />
+  <joint name="taotong_tool_joint" type="fixed">
+    <origin xyz="0 0 0" rpy="0 3.14 0" />
     <parent link="rokae_link7"/>
     <child link="tool_base_link"/>
   </joint>
-<!-- 手臂相机 -->
   <joint name="location_camera_joint" type="fixed">
-    <origin xyz="0.1 0 0" rpy="0 1.57 0"/>
-    <parent link="tool_base_link"/>
+    <origin xyz="0 0.15 1.75" rpy="0 3.14 1.57"/>
+    <parent link="rokae_link7"/>
     <child link="world_base"/>
   </joint>
-    <!-- <origin xyz="-0.40 0 -1.75" rpy="0 0 0"/> -->
-    <!-- <origin xyz="-0.25 0 -1.75" rpy="0 0 0"/> -->
 </robot>

Commit message: two camer add to scene  by per

File: rokae/src/realsense-ros-development/realsense2_description/urdf/test_d435_camera.urdf.xacro (robot description, xacro)
@@ -9,6 +9,6 @@
     </joint>
   <xacro:sensor_d435 name="camera" topics_ns="camera" parent="base_link" publish_pointcloud="true">
-    <origin xyz="0.25 0 1.75" rpy="0 1.57 0"/>
-    <!-- <origin xyz="0 0 0" rpy="0 0 0"/> -->
+    <!-- <origin xyz="0.25 0 1.75" rpy="0 1.57 0"/> -->
+    <origin xyz="0 0 0" rpy="0 0 0"/>
   </xacro:sensor_d435>
 </robot>
