Commit message: add battery_pack

File: rokae/src/cai_env/urdf/battery_pack.xacro (robot description, xacro)
@@ -48,5 +48,5 @@
   </link>
   <gazebo reference="battery_pack_link">
-        <material>Gazebo/Block</material>
+        <material>Gazebo/Black</material>
    </gazebo>
 <!-- luoshuan_Link -->

File: rokae/src/rokae_desk/urdf/robot.xacro (robot description, xacro)
@@ -52,5 +52,5 @@
   </transmission>
   <gazebo reference="${nameofManipulator}_base">
-     <material>Gazebo/Block</material>
+     <material>Gazebo/Black</material>
   </gazebo>
 <!--link 1-->
@@ -93,5 +93,5 @@
   </transmission>
   <gazebo reference="${nameofManipulator}_link1">
-     <material>Gazebo/Block</material>
+     <material>Gazebo/Black</material>
   </gazebo>
 <!--link 2-->
@@ -134,5 +134,5 @@
   </transmission>
   <gazebo reference="${nameofManipulator}_link2">
-     <material>Gazebo/Block</material>
+     <material>Gazebo/Black</material>
   </gazebo>
 <!--${nameofManipulator}_link 3-->
@@ -177,5 +177,5 @@
   </transmission>
   <gazebo reference="${nameofManipulator}_link3">
-     <material>Gazebo/Block</material>
+     <material>Gazebo/Black</material>
   </gazebo>
 <!--link 4-->
@@ -218,5 +218,5 @@
   </transmission>
   <gazebo reference="${nameofManipulator}_link4">
-     <material>Gazebo/Block</material>
+     <material>Gazebo/Black</material>
   </gazebo>
 <!--link 5-->
@@ -259,5 +259,5 @@
   </transmission>
   <gazebo reference="${nameofManipulator}_link5">
-     <material>Gazebo/Block</material>
+     <material>Gazebo/Black</material>
   </gazebo>
 <!--link 6-->
@@ -300,5 +300,5 @@
   </transmission>
   <gazebo reference="${nameofManipulator}_link6">
-     <material>Gazebo/Block</material>
+     <material>Gazebo/Black</material>
   </gazebo>
 <!--link 7-->
@@ -343,5 +343,5 @@
   </transmission> -->
   <gazebo reference="${nameofManipulator}_link7">
-     <material>Gazebo/Block</material>
+     <material>Gazebo/Black</material>
   </gazebo>
 <!-- ros_control plugin -->

File: rokae/src/rokae_desk/urdf/robot_tool.xacro (robot description, xacro)
@@ -52,5 +52,5 @@
   </transmission>
   <gazebo reference="${nameofManipulator}_base">
-     <material>Gazebo/Block</material>
+     <material>Gazebo/Black</material>
   </gazebo>
 <!--link 1-->
@@ -93,5 +93,5 @@
   </transmission>
   <gazebo reference="${nameofManipulator}_link1">
-     <material>Gazebo/Block</material>
+     <material>Gazebo/Black</material>
   </gazebo>
 <!--link 2-->
@@ -134,5 +134,5 @@
   </transmission>
   <gazebo reference="${nameofManipulator}_link2">
-     <material>Gazebo/Block</material>
+     <material>Gazebo/Black</material>
   </gazebo>
 <!--${nameofManipulator}_link 3-->
@@ -177,5 +177,5 @@
   </transmission>
   <gazebo reference="${nameofManipulator}_link3">
-     <material>Gazebo/Block</material>
+     <material>Gazebo/Black</material>
   </gazebo>
 <!--link 4-->
@@ -218,5 +218,5 @@
   </transmission>
   <gazebo reference="${nameofManipulator}_link4">
-     <material>Gazebo/Block</material>
+     <material>Gazebo/Black</material>
   </gazebo>
 <!--link 5-->
@@ -259,5 +259,5 @@
   </transmission>
   <gazebo reference="${nameofManipulator}_link5">
-     <material>Gazebo/Block</material>
+     <material>Gazebo/Black</material>
   </gazebo>
 <!--link 6-->
@@ -300,5 +300,5 @@
   </transmission>
   <gazebo reference="${nameofManipulator}_link6">
-     <material>Gazebo/Block</material>
+     <material>Gazebo/Black</material>
   </gazebo>
 <!--link 7-->
@@ -342,5 +342,5 @@
    -->
   <gazebo reference="${nameofManipulator}_link7">
-     <material>Gazebo/Block</material>
+     <material>Gazebo/Black</material>
   </gazebo>
 <!--tool -->

File: rokae/src/rokae_desk/urdf/robot_tool_complex.xacro (robot description, xacro)
@@ -3,5 +3,5 @@
   <xacro:include filename="$(find rokae_desk)/urdf/robot.xacro" />
   <xacro:include filename="$(find cai_env)/urdf/table.urdf.xacro" />
-  <xacro:include filename="$(find rokae_desk)/urdf/battery_pack.urdf" />
+  <xacro:include filename="$(find battery_pack_describe)/urdf/battery_pack.xacro" />
   <xacro:include filename="$(find rokae_desk)/urdf/camera_taotong.urdf" />
   <xacro:include filename="$(find realsense2_description)/urdf/test_d435_camera.urdf.xacro"   />

File: rokae/src/rokae_desk/urdf/rokae_robot.xacro (robot description, xacro)
@@ -52,5 +52,5 @@
   </transmission>
   <gazebo reference="${nameofManipulator}_base">
-     <material>Gazebo/Block</material>
+     <material>Gazebo/Black</material>
   </gazebo>
 <!--link 1-->
@@ -93,5 +93,5 @@
   </transmission>
   <gazebo reference="${nameofManipulator}_link1">
-     <material>Gazebo/Block</material>
+     <material>Gazebo/Black</material>
   </gazebo>
 <!--link 2-->
@@ -134,5 +134,5 @@
   </transmission>
   <gazebo reference="${nameofManipulator}_link2">
-     <material>Gazebo/Block</material>
+     <material>Gazebo/Black</material>
   </gazebo>
 <!--${nameofManipulator}_link 3-->
@@ -177,5 +177,5 @@
   </transmission>
   <gazebo reference="${nameofManipulator}_link3">
-     <material>Gazebo/Block</material>
+     <material>Gazebo/Black</material>
   </gazebo>
 <!--link 4-->
@@ -218,5 +218,5 @@
   </transmission>
   <gazebo reference="${nameofManipulator}_link4">
-     <material>Gazebo/Block</material>
+     <material>Gazebo/Black</material>
   </gazebo>
 <!--link 5-->
@@ -259,5 +259,5 @@
   </transmission>
   <gazebo reference="${nameofManipulator}_link5">
-     <material>Gazebo/Block</material>
+     <material>Gazebo/Black</material>
   </gazebo>
 <!--link 6-->
@@ -300,5 +300,5 @@
   </transmission>
   <gazebo reference="${nameofManipulator}_link6">
-     <material>Gazebo/Block</material>
+     <material>Gazebo/Black</material>
   </gazebo>
 <!--link 7-->
@@ -341,5 +341,5 @@
   </transmission>
   <gazebo reference="${nameofManipulator}_link7">
-     <material>Gazebo/Block</material>
+     <material>Gazebo/Black</material>
   </gazebo>
 <!--link 8-->
