Commit message: test  dask

File: rokae/src/cai_env/urdf/table.urdf.xacro (robot description, xacro)
@@ -31,5 +31,5 @@
       <geometry>
         <mesh
-          filename="package://cai_env/meshes/table.dae" />
+          filename="package://cai_env/meshes/desk_blender.dae" />
       </geometry>
     </visual>
@@ -40,10 +40,10 @@
       <geometry>
         <mesh
-          filename="package://cai_env/meshes/table.dae" />
+          filename="package://cai_env/meshes/desk_blender.dae" />
       </geometry>
     </collision>
-  <gazebo reference="table">
-    <material>Gazebo/WoodFloor</material>
-  </gazebo>
+      <!-- <gazebo reference="table">
+        <material>Gazebo/Green </material>
+      </gazebo>  -->
   </link>
 </robot>
