Commit message: 垂直的电池

File: rokae/src/battery_pack_describe/urdf/v_battery.urdf (robot description, URDF)
Before this commit: robot battery_pack_describe, 3 links, 2 joints
Links:
- removed link tilt_base_link
- removed link tilt_bolt_Link
- removed link tilt_nut_Link
- added link v_battery_base_link, mass 2.1452; collision mesh filename=package://battery_pack_describe/meshes/v_battery_base_link.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; visual mesh filename=package://battery_pack_describe/meshes/v_battery_base_link.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
- added link v_battery_bolt_Link, mass 0.010043058879212; collision mesh filename=package://battery_pack_describe/meshes/v_battery_bolt_Link.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; visual mesh filename=package://battery_pack_describe/meshes/v_battery_bolt_Link.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
- added link v_battery_nut_Link, mass 0.00265736664598247; collision mesh filename=package://battery_pack_describe/meshes/v_battery_nut_Link.S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; visual mesh filename=package://battery_pack_describe/meshes/v_battery_nut_Link.S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
Joints:
- removed joint tilt_bolt_joint
- removed joint tilt_nut_joint
- added joint v_battery_bolt_joint: type continuous, parent v_battery_base_link, child v_battery_bolt_Link, origin xyz=0.057323 -0.038452 0 rpy=0.39309 1.5708 0, axis 1 0 0
- added joint v_battery_nut_joint: type fixed, parent v_battery_base_link, child v_battery_nut_Link, origin xyz=0.057323 -0.038452 0 rpy=0 0 2.7485, axis 0 0 -1
