Commit message: for concept demo
1. adjust the color
2. add a script

File: rokae/src/battery_pack_describe/urdf/battery_pack.xacro (robot description, xacro)
@@ -87,9 +87,9 @@
   </link>
       <gazebo reference="bolt_vertical_Link">
-    <material>gazebo/editor</material>
+    <material>Gazebo/Grey</material>
   </gazebo>
   <joint
     name="bolt_vertical"
-    type="continuous">
+    type="fixed">
     <origin
       xyz="0.057323 -0.038452 0"
@@ -148,5 +148,5 @@
   </link>
   <gazebo reference="nut_vertical_Link">
-    <material>gazebo/editor</material>
+    <material>Gazebo/Grey</material>
   </gazebo>
   <joint
@@ -204,5 +204,5 @@
   </link>
   <gazebo reference="bolt_Horizontal_Link">
-    <material>gazebo/editor</material>
+    <material>Gazebo/Grey</material>
   </gazebo>
   <joint
@@ -260,5 +260,5 @@
   </link>
   <gazebo reference="nut_Horizontal_Link">
-    <material>gazebo/editor</material>
+    <material>Gazebo/Grey</material>
   </gazebo>
   <joint
@@ -316,5 +316,5 @@
   </link>
   <gazebo reference="bolt_Arbitrary_Link">
-    <material>gazebo/editor</material>
+    <material>Gazebo/Grey</material>
   </gazebo>
   <joint
@@ -372,5 +372,5 @@
   </link>
   <gazebo reference="nut_Sink_Link">
-    <material>gazebo/editor</material>
+    <material>Gazebo/Grey</material>
   </gazebo>
   <joint
@@ -428,5 +428,5 @@
   </link>
   <gazebo reference="bolt_Sink_Link">
-    <material>gazebo/editor</material>
+    <material>Gazebo/Grey</material>
   </gazebo>
   <joint
