Commit message: load battery to scene

File: rokae/src/battery_pack_describe/urdf/h_battery.urdf (robot description, URDF)
Before this commit: robot battery_pack_describe, 3 links, 2 joints
Links:
- removed link h_bolt__Link
- added link h_bolt_Link, mass 0.010043058879212; collision mesh filename=package://battery_pack_describe/meshes/h_bolt_Link.STL; visual mesh filename=package://battery_pack_describe/meshes/h_bolt_Link.STL
Joints:
- joint h_bolt_joint: child h_bolt__Link -> h_bolt_Link

File: rokae/src/battery_pack_describe/urdf/tilt_battery.urdf (robot description, URDF)
Before this commit: robot battery_pack_describe, 3 links, 2 joints
Joints:
- joint tilt_nut_joint: type fixed -> continuous

File: rokae/src/rokae_desk/urdf/camera_taotong.urdf (robot description, URDF)
Before this commit: robot rokea, 2 links, 1 joints
Links:
- link tool_link: geometry collision mesh filename=package://rokae_desk/meshes/tool_Link.stl; visual mesh filename=package://rokae_desk/meshes/tool_Link.stl scale=1.7 1.7 1.7

File: rokae/src/rokae_desk/urdf/robot_tool_complex.xacro (robot description, xacro)
@@ -3,5 +3,5 @@
   <xacro:include filename="$(find rokae_desk)/urdf/robot.xacro" />
   <xacro:include filename="$(find cai_env)/urdf/table.urdf.xacro" />
-  <xacro:include filename="$(find battery_pack_describe)/urdf/battery_pack.xacro" />
+  <!-- <xacro:include filename="$(find battery_pack_describe)/urdf/battery_pack.xacro" /> -->
   <xacro:include filename="$(find rokae_desk)/urdf/camera_taotong.urdf" />
   <xacro:include filename="$(find realsense2_description)/urdf/test_d435_camera.urdf.xacro"   />
@@ -18,9 +18,9 @@
     <child link="rokae_base"/>
   </joint>
-  <joint name="battery_pack_joint" type="fixed">
+  <!-- <joint name="battery_pack_joint" type="fixed">
     <origin xyz="0 0 0.12" rpy="0 0 3.14" />
     <parent link="table"/>
     <child link="battery_pack_link"/>
-  </joint>
+  </joint> -->
   <joint name="taotong_tool_joint" type="fixed">
     <origin xyz="0 0 0" rpy="0 3.14 0" />

Commit message: 其它电池纹理修改

File: rokae/src/battery_pack_describe/urdf/h_battery.urdf (robot description, URDF)
Before this commit: robot battery_pack_describe, 3 links, 2 joints
Links:
- link h_battery_base_link: geometry collision mesh filename=package://battery_pack_describe/meshes/v_battery_base_link.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; visual mesh filename=package://battery_pack_describe/meshes/v_battery_base_link.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

File: rokae/src/battery_pack_describe/urdf/h_battery.xacro (robot description, xacro)
@@ -26,5 +26,5 @@
       <geometry>
         <mesh
-          filename="package://battery_pack_describe/meshes/h_battery_base_link.STL" />
+        <mesh filename="package://battery_pack_describe/meshes/v_battery_base_link.dae"/>
       </geometry>
       <material
@@ -40,11 +40,13 @@
       <geometry>
         <mesh
-          filename="package://battery_pack_describe/meshes/h_battery_base_link.STL" />
+        <mesh filename="package://battery_pack_describe/meshes/v_battery_base_link.dae"/>
       </geometry>
     </collision>
   </link>
+<!--
       <gazebo reference="h_battery_base_link">
     <material>Gazebo/FlatBlack</material>
   </gazebo>
+ -->
   <link
     name="h_bolt_Link">

File: rokae/src/battery_pack_describe/urdf/hole_battery.urdf (robot description, URDF)
Before this commit: robot hole_battery_describe, 3 links, 2 joints
Links:
- link hole_base_link: geometry collision mesh filename=package://battery_pack_describe/meshes/hole_base_link.dae; visual mesh filename=package://battery_pack_describe/meshes/hole_base_link.dae

File: rokae/src/battery_pack_describe/urdf/hole_battery.xacro (robot description, xacro)
@@ -26,5 +26,5 @@
       <geometry>
         <mesh
-          filename="package://battery_pack_describe/meshes/hole_base_link.STL" />
+          filename="package://battery_pack_describe/meshes/hole_base_link.dae" />
       </geometry>
       <material
@@ -40,11 +40,11 @@
       <geometry>
         <mesh
-          filename="package://battery_pack_describe/meshes/hole_base_link.STL" />
+          filename="package://battery_pack_describe/meshes/hole_base_link.dae" />
       </geometry>
     </collision>
   </link>
-      <gazebo reference="hole_base_link">
+      <!-- <gazebo reference="hole_base_link">
     <material>Gazebo/FlatBlack</material>
-  </gazebo>
+  </gazebo> -->
   <link
     name="hole_bolt_Link">

File: rokae/src/battery_pack_describe/urdf/tilt_battery.urdf (robot description, URDF)
Before this commit: robot battery_pack_describe, 3 links, 2 joints
Links:
- link tilt_base_link: geometry collision mesh filename=package://battery_pack_describe/meshes/v_battery_base_link.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; visual mesh filename=package://battery_pack_describe/meshes/v_battery_base_link.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

File: rokae/src/battery_pack_describe/urdf/tilt_battery.xacro (robot description, xacro)
@@ -26,6 +26,5 @@
         rpy="0 0 0" />
       <geometry>
-        <mesh
-          filename="package://battery_pack_describe/meshes/tilt_base_link.STL" />
+        <mesh filename="package://battery_pack_describe/meshes/v_battery_base_link.dae"/>
       </geometry>
       <material
@@ -40,12 +39,12 @@
         rpy="0 0 0" />
       <geometry>
-        <mesh
-          filename="package://battery_pack_describe/meshes/tilt_base_link.STL" />
+        <mesh filename="package://battery_pack_describe/meshes/v_battery_base_link.dae"/>
       </geometry>
     </collision>
   </link>
+<!--
       <gazebo reference="tilt_base_link">
     <material>Gazebo/FlatBlack</material>
-  </gazebo>
+  </gazebo> -->
   <link
     name="tilt_bolt_Link">
