Commit message: edit color

File: rokae/src/battery_pack_describe/urdf/h_battery.xacro (robot description, xacro)
@@ -91,4 +91,10 @@
       <gazebo reference="h_bolt_Link">
     <material>Gazebo/Gray</material>
+        <mu1>100.0</mu1>
+	    <mu2>100.0</mu2>
+	    <kp>1000000.0</kp>
+	    <kd>100.0</kd>
+	    <minDepth>0.001</minDepth>
+	    <maxVel>1.0</maxVel>
   </gazebo>
   <joint

File: rokae/src/battery_pack_describe/urdf/hole_battery.xacro (robot description, xacro)
@@ -89,4 +89,10 @@
       <gazebo reference="hole_bolt_Link">
     <material>Gazebo/Gray</material>
+        <mu1>100.0</mu1>
+	    <mu2>100.0</mu2>
+	    <kp>1000000.0</kp>
+	    <kd>100.0</kd>
+	    <minDepth>0.001</minDepth>
+	    <maxVel>1.0</maxVel>
   </gazebo>
   <joint

File: rokae/src/battery_pack_describe/urdf/tilt_battery.xacro (robot description, xacro)
@@ -89,4 +89,10 @@
       <gazebo reference="tilt_bolt_Link">
     <material>Gazebo/Gray</material>
+        <mu1>100.0</mu1>
+	    <mu2>100.0</mu2>
+	    <kp>1000000.0</kp>
+	    <kd>100.0</kd>
+	    <minDepth>0.001</minDepth>
+	    <maxVel>1.0</maxVel>
   </gazebo>
   <joint

File: rokae/src/battery_pack_describe/urdf/v_battery.xacro (robot description, xacro)
@@ -44,11 +44,13 @@
   </link>
   <gazebo reference="v_battery_base_link">
-    <mu1>0.1</mu1>
-    <mu2>0.1</mu2>
-    <kp>1</kp>
-    <kd>500.0</kd>
-    <minDepth>0.001</minDepth>
+    <mu1>10.0</mu1>
+	    <mu2>10.0</mu2>
+	    <kp>1000000.0</kp>
+	    <kd>100.0</kd>
+	    <minDepth>0.001</minDepth>
+	    <maxVel>1.0</maxVel>
+    <!-- <minDepth>0.001</minDepth>
     <maxVel>0.1</maxVel>
-    <fdir1>1 0 0</fdir1>
+    <fdir1>1 0 0</fdir1> -->
   </gazebo>
   <link    name="v_battery_bolt_Link">
@@ -92,12 +94,14 @@
   </link>
   <gazebo reference="v_battery_bolt_Link">
-    <mu1>0.1</mu1>
-    <mu2>0.1</mu2>
-    <kp>1</kp>
-    <kd>10.0</kd>
-    <minDepth>0.001</minDepth>
+    <mu1>100.0</mu1>
+	    <mu2>100.0</mu2>
+	    <kp>1000000.0</kp>
+	    <kd>100.0</kd>
+	    <minDepth>0.001</minDepth>
+	    <maxVel>1.0</maxVel>
+    <!-- <minDepth>0.001</minDepth>
     <maxVel>0.1</maxVel>
-    <fdir1>1 0 0</fdir1>
-    <material>Gazebo/FlatBlack</material>
+    <fdir1>1 0 0</fdir1> -->
+    <material>Gazebo/Black</material>
 </gazebo>
   <joint

File: rokae/src/cai_env/urdf/table.urdf.xacro (robot description, xacro)
@@ -43,4 +43,7 @@
       </geometry>
     </collision>
+  <gazebo reference="table">
+    <material>Gazebo/WoodFloor</material>
+  </gazebo>
   </link>
 </robot>

Commit message: 改善电池包加载方式和纠正了错误

File: rokae/src/battery_pack_describe/urdf/h_battery.xacro (robot description, xacro)
@@ -25,6 +25,5 @@
         rpy="0 0 0" />
       <geometry>
-        <mesh
-        <mesh filename="package://battery_pack_describe/meshes/v_battery_base_link.dae"/>
+        <mesh     filename="package://battery_pack_describe/meshes/v_battery_base_link.dae" />
       </geometry>
       <material
@@ -39,6 +38,5 @@
         rpy="0 0 0" />
       <geometry>
-        <mesh
-        <mesh filename="package://battery_pack_describe/meshes/v_battery_base_link.dae"/>
+        <mesh     filename="package://battery_pack_describe/meshes/v_battery_base_link.dae" />
       </geometry>
     </collision>

File: rokae/src/cai_env/urdf/table.urdf.xacro (robot description, xacro)
@@ -31,5 +31,5 @@
       <geometry>
         <mesh
-          filename="package://cai_env/meshes/desk_blender.dae" />
+          filename="package://cai_env/meshes/table_blend.dae" />
       </geometry>
     </visual>
@@ -40,10 +40,10 @@
       <geometry>
         <mesh
-          filename="package://cai_env/meshes/desk_blender.dae" />
+          filename="package://cai_env/meshes/table_blend.dae" />
       </geometry>
     </collision>
-      <!-- <gazebo reference="table">
-        <material>Gazebo/Green </material>
-      </gazebo>  -->
+    <gazebo reference="table">
+      <material>Gazebo/Green </material>
+    </gazebo>
   </link>
 </robot>

Commit message: 修改电池包

File: rokae/src/battery_pack_describe/urdf/h_battery.xacro (robot description, xacro)
@@ -87,12 +87,13 @@
     </collision>
   </link>
-      <gazebo reference="h_bolt_Link">
+  <gazebo reference="h_bolt_Link">
     <material>Gazebo/Gray</material>
-        <mu1>100.0</mu1>
-	    <mu2>100.0</mu2>
-	    <kp>1000000.0</kp>
-	    <kd>100.0</kd>
-	    <minDepth>0.001</minDepth>
-	    <maxVel>1.0</maxVel>
+    <mu1>10.0</mu>
+    <mu2>10.0</mu2>
+    <kp>1000000.0</kp>
+    <kd>100.0</kd>
+    <minDepth>0.001</minDepth>
+    <maxVel>1.0</maxVel>
+    <fdir1>1 0 0</fdir1>
   </gazebo>
   <joint

File: rokae/src/battery_pack_describe/urdf/hole_battery.xacro (robot description, xacro)
@@ -87,12 +87,13 @@
     </collision>
   </link>
-      <gazebo reference="hole_bolt_Link">
+  <gazebo reference="hole_bolt_Link">
     <material>Gazebo/Gray</material>
-        <mu1>100.0</mu1>
-	    <mu2>100.0</mu2>
-	    <kp>1000000.0</kp>
-	    <kd>100.0</kd>
-	    <minDepth>0.001</minDepth>
-	    <maxVel>1.0</maxVel>
+    <mu1>10.0</mu>
+    <mu2>10.0</mu2>
+    <kp>1000000.0</kp>
+    <kd>100.0</kd>
+    <minDepth>0.001</minDepth>
+    <maxVel>1.0</maxVel>
+    <fdir1>1 0 0</fdir1>
   </gazebo>
   <joint

File: rokae/src/battery_pack_describe/urdf/tilt_battery.xacro (robot description, xacro)
@@ -87,12 +87,13 @@
     </collision>
   </link>
-      <gazebo reference="tilt_bolt_Link">
+  <gazebo reference="tilt_bolt_Link">
     <material>Gazebo/Gray</material>
-        <mu1>100.0</mu1>
-	    <mu2>100.0</mu2>
-	    <kp>1000000.0</kp>
-	    <kd>100.0</kd>
-	    <minDepth>0.001</minDepth>
-	    <maxVel>1.0</maxVel>
+    <mu1>10.0</mu>
+    <mu2>10.0</mu2>
+    <kp>1000000.0</kp>
+    <kd>100.0</kd>
+    <minDepth>0.001</minDepth>
+    <maxVel>1.0</maxVel>
+    <fdir1>1 0 0</fdir1>
   </gazebo>
   <joint

File: rokae/src/battery_pack_describe/urdf/v_battery.xacro (robot description, xacro)
@@ -75,8 +75,7 @@
       <geometry>
         <mesh
-          filename="package://battery_pack_describe/meshes/v_battery_bolt_Link.dae" />
+          filename="package://battery_pack_describe/meshes/v_battery_bolt_Link_metal.dae" />
       </geometry>
-      <material
-        name="">
+      <material  name="">
         <color
           rgba="0.776470588235294 0.756862745098039 0.737254901960784 1" />
@@ -89,5 +88,5 @@
       <geometry>
         <mesh
-          filename="package://battery_pack_describe/meshes/v_battery_bolt_Link.dae" />
+          filename="package://battery_pack_describe/meshes/v_battery_bolt_Link_metal.dae" />
       </geometry>
     </collision>

File: rokae/src/rokae_desk/urdf/robot_tool_complex.xacro (robot description, xacro)
@@ -4,5 +4,5 @@
   <xacro:include filename="$(find cai_env)/urdf/table.urdf.xacro" />
   <!-- <xacro:include filename="$(find battery_pack_describe)/urdf/battery_pack.xacro" /> -->
-  <xacro:include filename="$(find rokae_desk)/urdf/camera_taotong.urdf" />
+  <xacro:include filename="$(find rokae_desk)/urdf/camera_taotong.xacro" />
   <xacro:include filename="$(find realsense2_description)/urdf/test_d435_camera.urdf.xacro"   />
   <xacro:include filename="$(find realsense2_description)/urdf/gloal_d435_camera.urdf.xacro"   />

Commit message: 修改了螺栓的自转问题，电池包也会自转，我在测试测试

File: rokae/src/battery_pack_describe/urdf/h_battery.xacro (robot description, xacro)
@@ -42,9 +42,14 @@
     </collision>
   </link>
-<!--
-      <gazebo reference="h_battery_base_link">
-    <material>Gazebo/FlatBlack</material>
+  <gazebo reference="h_battery_base_link">
+      <maxVel>0.01</maxVel>
+      <kd>1</kd>
+      <maxContacts>20</maxContacts>
+      <mu2>50000</mu2>
+      <selfCollide>0</selfCollide>
+      <mu1>50000</mu1>
+      <minDepth>0</minDepth>
+      <kp>1000000000000.0</kp>
   </gazebo>
- -->
   <link
     name="h_bolt_Link">
@@ -88,12 +93,13 @@
   </link>
   <gazebo reference="h_bolt_Link">
-    <material>Gazebo/Gray</material>
-    <mu1>10.0</mu>
-    <mu2>10.0</mu2>
-    <kp>1000000.0</kp>
-    <kd>100.0</kd>
-    <minDepth>0.001</minDepth>
-    <maxVel>1.0</maxVel>
-    <fdir1>1 0 0</fdir1>
+      <maxVel>0.01</maxVel>
+      <kd>1</kd>
+      <maxContacts>20</maxContacts>
+      <mu2>50000</mu2>
+      <selfCollide>0</selfCollide>
+      <mu1>50000</mu1>
+      <minDepth>0</minDepth>
+      <kp>1000000000000.0</kp>
+    <material>Gazebo/Grey </material>
   </gazebo>
   <joint

File: rokae/src/battery_pack_describe/urdf/hole_battery.xacro (robot description, xacro)
@@ -44,7 +44,15 @@
     </collision>
   </link>
-      <!-- <gazebo reference="hole_base_link">
-    <material>Gazebo/FlatBlack</material>
-  </gazebo> -->
+  <gazebo reference="hole_base_link">
+    <!-- <material>Gazebo/FlatBlack</material> -->
+      <maxVel>0.01</maxVel>
+      <kd>1</kd>
+      <maxContacts>20</maxContacts>
+      <mu2>50000</mu2>
+      <selfCollide>0</selfCollide>
+      <mu1>50000</mu1>
+      <minDepth>0</minDepth>
+      <kp>1000000000000.0</kp>
+  </gazebo>
   <link
     name="hole_bolt_Link">
@@ -88,12 +96,13 @@
   </link>
   <gazebo reference="hole_bolt_Link">
-    <material>Gazebo/Gray</material>
-    <mu1>10.0</mu>
-    <mu2>10.0</mu2>
-    <kp>1000000.0</kp>
-    <kd>100.0</kd>
-    <minDepth>0.001</minDepth>
-    <maxVel>1.0</maxVel>
-    <fdir1>1 0 0</fdir1>
+      <maxVel>0.01</maxVel>
+      <kd>1</kd>
+      <maxContacts>20</maxContacts>
+      <mu2>50000</mu2>
+      <selfCollide>0</selfCollide>
+      <mu1>50000</mu1>
+      <minDepth>0</minDepth>
+      <kp>1000000000000.0</kp>
+    <material>Gazebo/Grey </material>
   </gazebo>
   <joint

File: rokae/src/battery_pack_describe/urdf/tilt_battery.xacro (robot description, xacro)
@@ -43,8 +43,15 @@
     </collision>
   </link>
-<!--
-      <gazebo reference="tilt_base_link">
-    <material>Gazebo/FlatBlack</material>
-  </gazebo> -->
+  <gazebo reference="tilt_base_link">
+    <!-- <material>Gazebo/FlatBlack</material> -->
+      <maxVel>0.01</maxVel>
+      <kd>1</kd>
+      <maxContacts>20</maxContacts>
+      <mu2>50000</mu2>
+      <selfCollide>0</selfCollide>
+      <mu1>50000</mu1>
+      <minDepth>0</minDepth>
+      <kp>1000000000000.0</kp>
+  </gazebo>
   <link
     name="tilt_bolt_Link">
@@ -87,13 +94,15 @@
     </collision>
   </link>
+<!--摩擦力参考链接，我修改了mu的大小。https://daimajiaoliu.com/daima/48713c82b900404。 http://blog.robotakao.jp/blog-entry-441.html -->
   <gazebo reference="tilt_bolt_Link">
-    <material>Gazebo/Gray</material>
-    <mu1>10.0</mu>
-    <mu2>10.0</mu2>
-    <kp>1000000.0</kp>
-    <kd>100.0</kd>
-    <minDepth>0.001</minDepth>
-    <maxVel>1.0</maxVel>
-    <fdir1>1 0 0</fdir1>
+      <maxVel>0.01</maxVel>
+      <kd>1</kd>
+      <maxContacts>20</maxContacts>
+      <mu2>50000</mu2>
+      <selfCollide>0</selfCollide>
+      <mu1>50000</mu1>
+      <minDepth>0</minDepth>
+      <kp>1000000000000.0</kp>
+    <material>Gazebo/Grey </material>
   </gazebo>
   <joint

File: rokae/src/battery_pack_describe/urdf/v_battery.xacro (robot description, xacro)
@@ -44,13 +44,12 @@
   </link>
   <gazebo reference="v_battery_base_link">
-    <mu1>10.0</mu1>
-	    <mu2>10.0</mu2>
-	    <kp>1000000.0</kp>
-	    <kd>100.0</kd>
-	    <minDepth>0.001</minDepth>
-	    <maxVel>1.0</maxVel>
-    <!-- <minDepth>0.001</minDepth>
-    <maxVel>0.1</maxVel>
-    <fdir1>1 0 0</fdir1> -->
+      <maxVel>0.01</maxVel>
+      <kd>1</kd>
+      <maxContacts>20</maxContacts>
+      <mu2>500000</mu2>
+      <selfCollide>0</selfCollide>
+      <mu1>500000</mu1>
+      <minDepth>0</minDepth>
+      <kp>1000000000000.0</kp>
   </gazebo>
   <link    name="v_battery_bolt_Link">
@@ -92,14 +91,16 @@
     </collision>
   </link>
+<!--摩擦力参考链接，我修改了mu的大小。 https://boschresearch.github.io/pcg_gazebo_pkgs/tutorials/parsers/urdf/robots/
+https://whtqh.gitbooks.io/gazebo_simu_chs/content/using_a_urdf_model.html  摩擦力和其他参数，定义链接
+-->
   <gazebo reference="v_battery_bolt_Link">
-    <mu1>1000.0</mu1>
-	    <mu2>1000.0</mu2>
-	    <kp>1000000.0</kp>
-	    <kd>100.0</kd>
-	    <minDepth>0.001</minDepth>
-	    <maxVel>1.0</maxVel>
-    <!-- <minDepth>0.001</minDepth>
-    <maxVel>0.1</maxVel>
-    <fdir1>1 0 0</fdir1> -->
+      <maxVel>0.01</maxVel>
+      <kd>1</kd>
+      <maxContacts>20</maxContacts>
+      <mu2>50000</mu2>
+      <selfCollide>0</selfCollide>
+      <mu1>50000</mu1>
+      <minDepth>0</minDepth>
+      <kp>1000000000000.0</kp>
     <material>Gazebo/Grey </material>
 </gazebo>

Commit message: 电池包添加碰撞盒

File: rokae/src/battery_pack_describe/urdf/h_battery.xacro (robot description, xacro)
@@ -38,4 +38,5 @@
         rpy="0 0 0" />
       <geometry>
+        <box size="0.5 0.5 0.05" />
         <mesh     filename="package://battery_pack_describe/meshes/v_battery_base_link.dae" />
       </geometry>
@@ -87,4 +88,5 @@
         rpy="0 0 0" />
       <geometry>
+        <cylinder length="0.04" radius="0.02"/>
         <mesh
           filename="package://battery_pack_describe/meshes/h_bolt_Link.STL" />

File: rokae/src/battery_pack_describe/urdf/hole_battery.xacro (robot description, xacro)
@@ -39,4 +39,5 @@
         rpy="0 0 0" />
       <geometry>
+        <box size="0.5 0.5 0.05" />
         <mesh
           filename="package://battery_pack_describe/meshes/hole_base_link.dae" />
@@ -90,4 +91,5 @@
         rpy="0 0 0" />
       <geometry>
+        <cylinder length="0.04" radius="0.02"/>
         <mesh
           filename="package://battery_pack_describe/meshes/hole_bolt_Link.STL" />

File: rokae/src/battery_pack_describe/urdf/tilt_battery.xacro (robot description, xacro)
@@ -39,4 +39,5 @@
         rpy="0 0 0" />
       <geometry>
+         <cylinder length="0.1" radius="0.02"/>
         <mesh filename="package://battery_pack_describe/meshes/v_battery_base_link.dae"/>
       </geometry>
@@ -96,4 +97,5 @@
         rpy="0 0 0" />
       <geometry>
+        <box size="0.5 0.5 0.05" />
         <mesh
           filename="package://battery_pack_describe/meshes/tilt_bolt_Link.STL" />

File: rokae/src/battery_pack_describe/urdf/v_battery.xacro (robot description, xacro)
@@ -6,9 +6,6 @@
   <link    name="v_battery_base_link"  xmlns:xacro="http://www.ros.org/wiki/xacro">
     <inertial>
-      <origin
-        xyz="-0.17823 0.0014541 -0.18254"
-        rpy="0 0 0" />
-      <mass
-        value="2.1452" />
+      <origin   xyz="-0.17823 0.0014541 -0.18254"  rpy="0 0 0" />
+      <mass        value="2.1452" />
       <inertia
         ixx="0.04437"
@@ -20,21 +17,16 @@
     </inertial>
     <visual>
-      <origin
-        xyz="0 0 0"
-        rpy="0 0 0" />
+      <origin   xyz="0 0 0"   rpy="0 0 0" />
       <geometry>
         <mesh     filename="package://battery_pack_describe/meshes/v_battery_base_link.dae" />
       </geometry>
-      <material
-        name="">
-        <color
-          rgba="0.79216 0.81961 0.93333 1" />
+      <material     name="">
+        <color    rgba="0.79216 0.81961 0.93333 1" />
       </material>
     </visual>
     <collision>
-      <origin
-        xyz="0 0 0"
-        rpy="0 0 0" />
+      <origin     xyz="0 0 0"    rpy="0 0 0" />
       <geometry>
+        <box size="0.5 0.5 0.05" />
         <mesh
           filename="package://battery_pack_describe/meshes/v_battery_base_link.dae" />
@@ -73,9 +65,7 @@
   <link    name="v_battery_bolt_Link">
     <inertial>
-      <origin
-        xyz="-0.00224797355412683 -2.42669320749123E-09 1.13997717515746E-09"
+      <origin     xyz="-0.00224797355412683 -2.42669320749123E-09 1.13997717515746E-09"
         rpy="0 0 0" />
-      <mass
-        value="0.010043058879212" />
+      <mass  value="0.010043058879212" />
       <inertia
         ixx="8.16036465000949E-08"
@@ -87,23 +77,17 @@
     </inertial>
     <visual>
-      <origin
-        xyz="0 0 0"
-        rpy="0 0 0" />
+      <origin   xyz="0 0 0"  rpy="0 0 0" />
       <geometry>
-        <mesh
-          filename="package://battery_pack_describe/meshes/v_battery_bolt_Link_metal.dae" />
+        <mesh   filename="package://battery_pack_describe/meshes/v_battery_bolt_Link_metal.dae" />
       </geometry>
       <material  name="">
-        <color
-          rgba="0.776470588235294 0.756862745098039 0.737254901960784 1" />
+        <color  rgba="0.776470588235294 0.756862745098039 0.737254901960784 1" />
       </material>
     </visual>
     <collision>
-      <origin
-        xyz="0 0 0"
-        rpy="0 0 0" />
+      <origin   xyz="0 0 0"   rpy="0 0 0" />
       <geometry>
-        <mesh
-          filename="package://battery_pack_describe/meshes/v_battery_bolt_Link_metal.dae" />
+        <cylinder length="0.1" radius="0.02"/>
+        <mesh   filename="package://battery_pack_describe/meshes/v_battery_bolt_Link_metal.dae" />
       </geometry>
     </collision>
@@ -153,24 +137,17 @@
     </inertial>
     <visual>
-      <origin
-        xyz="0 0 0"
-        rpy="0 0 0" />
+      <origin   xyz="0 0 0"  rpy="0 0 0" />
       <geometry>
-        <mesh
-          filename="package://battery_pack_describe/meshes/v_battery_nut_Link.dae" />
+        <mesh    filename="package://battery_pack_describe/meshes/v_battery_nut_Link.dae" />
       </geometry>
-      <material
-        name="">
-        <color
-          rgba="0.776470588235294 0.756862745098039 0.737254901960784 1" />
+      <material     name="">
+        <color    rgba="0.776470588235294 0.756862745098039 0.737254901960784 1" />
       </material>
     </visual>
     <collision>
-      <origin
-        xyz="0 0 0"
-        rpy="0 0 0" />
+      <origin        xyz="0 0 0"        rpy="0 0 0" />
       <geometry>
-        <mesh
-          filename="package://battery_pack_describe/meshes/v_battery_nut_Link.dae" />
+        <cylinder length="0.04" radius="0.02"/>
+        <mesh   filename="package://battery_pack_describe/meshes/v_battery_nut_Link.dae" />
       </geometry>
     </collision>
