Commit message: test

File: rokae/src/battery_pack_describe/urdf/v_battery.xacro (robot description, xacro)
@@ -44,5 +44,5 @@
   </link>
       <gazebo reference="v_battery_base_link">
-    <material>Gazebo/FlatBlack</material>
+    <material>Gazebo/LaserScan2nd</material>
   </gazebo>
   <link    name="v_battery_bolt_Link">
@@ -85,6 +85,6 @@
     </collision>
   </link>
-      <gazebo reference="v_battery_bolt_Link">
-    <material>Gazebo/Gray</material>
+  <gazebo reference="v_battery_bolt_Link">
+    <material>PR2/White </material>
   </gazebo>
   <joint

Commit message: v battery 模型渲染

File: rokae/src/battery_pack_describe/urdf/v_battery.xacro (robot description, xacro)
@@ -25,5 +25,5 @@
         rpy="0 0 0" />
       <geometry>
-        <mesh     filename="package://battery_pack_describe/meshes/v_battery_base_link.STL" />
+        <mesh     filename="package://battery_pack_describe/meshes/v_battery_base_link.dae" />
       </geometry>
       <material
@@ -39,11 +39,11 @@
       <geometry>
         <mesh
-          filename="package://battery_pack_describe/meshes/v_battery_base_link.STL" />
+          filename="package://battery_pack_describe/meshes/v_battery_base_link.dae" />
       </geometry>
     </collision>
   </link>
-      <gazebo reference="v_battery_base_link">
-    <material>Gazebo/LaserScan2nd</material>
-  </gazebo>
+      <!-- <gazebo reference="v_battery_base_link">
+    <material>Gazebo/FlatBlack</material>
+  </gazebo> -->
   <link    name="v_battery_bolt_Link">
     <inertial>
@@ -67,5 +67,5 @@
       <geometry>
         <mesh
-          filename="package://battery_pack_describe/meshes/v_battery_bolt_Link.STL" />
+          filename="package://battery_pack_describe/meshes/v_battery_bolt_Link.dae" />
       </geometry>
       <material
@@ -81,11 +81,12 @@
       <geometry>
         <mesh
-          filename="package://battery_pack_describe/meshes/v_battery_bolt_Link.STL" />
+          filename="package://battery_pack_describe/meshes/v_battery_bolt_Link.dae" />
       </geometry>
     </collision>
   </link>
-  <gazebo reference="v_battery_bolt_Link">
-    <material>PR2/White </material>
+      <!-- <gazebo reference="v_battery_bolt_Link">
+    <material>Gazebo/Gray</material>
   </gazebo>
+ -->
   <joint
     name="v_battery_bolt_joint"
@@ -123,5 +124,5 @@
       <geometry>
         <mesh
-          filename="package://battery_pack_describe/meshes/v_battery_nut_Link.STL" />
+          filename="package://battery_pack_describe/meshes/v_battery_nut_Link.dae" />
       </geometry>
       <material
@@ -137,11 +138,11 @@
       <geometry>
         <mesh
-          filename="package://battery_pack_describe/meshes/v_battery_nut_Link.STL" />
+          filename="package://battery_pack_describe/meshes/v_battery_nut_Link.dae" />
       </geometry>
     </collision>
   </link>
-  <gazebo reference="v_battery_nut_Link">
+  <!-- <gazebo reference="v_battery_nut_Link">
     <material>Gazebo/Gray</material>
-  </gazebo>
+  </gazebo> -->
   <joint
     name="v_battery_nut_joint"

Commit message: image position

File: rokae/src/battery_pack_describe/urdf/v_battery.xacro (robot description, xacro)
@@ -85,8 +85,7 @@
     </collision>
   </link>
-      <!-- <gazebo reference="v_battery_bolt_Link">
+  <gazebo reference="v_battery_bolt_Link">
     <material>Gazebo/Gray</material>
   </gazebo>
- -->
   <joint
     name="v_battery_bolt_joint"

File: rokae/src/rokae_desk/urdf/robot_tool_complex.xacro (robot description, xacro)
@@ -34,5 +34,5 @@
   </joint>
   <joint name="scene_camera_joint" type="fixed">
-    <origin xyz="0 0 1.75" rpy="0 1.57 1.57"/>
+    <origin xyz="0 0 1.55" rpy="0 1.57 1.57"/>
     <parent link="table"/>
     <child link="gloal_world_base"/>

Commit message: bolt color  and   other para

File: rokae/src/battery_pack_describe/urdf/v_battery.xacro (robot description, xacro)
@@ -43,7 +43,13 @@
     </collision>
   </link>
-      <!-- <gazebo reference="v_battery_base_link">
-    <material>Gazebo/FlatBlack</material>
-  </gazebo> -->
+  <gazebo reference="v_battery_base_link">
+    <mu1>0.1</mu1>
+    <mu2>0.1</mu2>
+    <kp>1</kp>
+    <kd>500.0</kd>
+    <minDepth>0.001</minDepth>
+    <maxVel>0.1</maxVel>
+    <fdir1>1 0 0</fdir1>
+  </gazebo>
   <link    name="v_battery_bolt_Link">
     <inertial>
@@ -86,6 +92,13 @@
   </link>
   <gazebo reference="v_battery_bolt_Link">
-    <material>Gazebo/Gray</material>
-  </gazebo>
+    <mu1>0.1</mu1>
+    <mu2>0.1</mu2>
+    <kp>1</kp>
+    <kd>10.0</kd>
+    <minDepth>0.001</minDepth>
+    <maxVel>0.1</maxVel>
+    <fdir1>1 0 0</fdir1>
+    <material>Gazebo/FlatBlack</material>
+</gazebo>
   <joint
     name="v_battery_bolt_joint"
@@ -141,7 +154,14 @@
     </collision>
   </link>
-  <!-- <gazebo reference="v_battery_nut_Link">
-    <material>Gazebo/Gray</material>
-  </gazebo> -->
+  <gazebo reference="v_battery_nut_Link">
+    <mu1>0.1</mu1>
+    <mu2>0.1</mu2>
+    <kp>1</kp>
+    <kd>10.0</kd>
+    <minDepth>0.001</minDepth>
+    <maxVel>0.1</maxVel>
+    <fdir1>1 0 0</fdir1>
+    <material>Gazebo/FlatBlack</material>
+  </gazebo>
   <joint
     name="v_battery_nut_joint"

Commit message: color

File: rokae/src/battery_pack_describe/urdf/v_battery.xacro (robot description, xacro)
@@ -94,6 +94,6 @@
   </link>
   <gazebo reference="v_battery_bolt_Link">
-    <mu1>100.0</mu1>
-	    <mu2>100.0</mu2>
+    <mu1>1000.0</mu1>
+	    <mu2>1000.0</mu2>
 	    <kp>1000000.0</kp>
 	    <kd>100.0</kd>
@@ -103,5 +103,5 @@
     <maxVel>0.1</maxVel>
     <fdir1>1 0 0</fdir1> -->
-    <material>Gazebo/Black</material>
+    <material>Gazebo/Grey </material>
 </gazebo>
   <joint

Commit message: 修改了电池包的摩擦系数，不好使，不能用重力，会出错

File: rokae/src/battery_pack_describe/urdf/v_battery.xacro (robot description, xacro)
@@ -44,12 +44,22 @@
   </link>
   <gazebo reference="v_battery_base_link">
-      <maxVel>0.01</maxVel>
-      <kd>1</kd>
-      <maxContacts>20</maxContacts>
-      <mu2>500000</mu2>
-      <selfCollide>0</selfCollide>
-      <mu1>500000</mu1>
-      <minDepth>0</minDepth>
+      <maxVel>100</maxVel>
+      <kd>200</kd>
+      <maxContacts>200</maxContacts>
+      <mu2>5000000000000</mu2>
+      <selfCollide>10</selfCollide>
+      <mu1>5000000000000</mu1>
+      <minDepth>10</minDepth>
       <kp>1000000000000.0</kp>
+      <!-- <gravity>bool</gravity> -->
+      <!-- <gravity>bool</gravity> -->
+      <!-- <maxVel>100</maxVel>
+      <kd>10</kd>
+      <maxContacts>200</maxContacts>
+      <mu2>10</mu2>
+      <selfCollide>10</selfCollide>
+      <mu1>10</mu1>
+      <minDepth>10</minDepth>
+      <kp>1</kp> -->
   </gazebo>
   <link    name="v_battery_bolt_Link">

File: rokae/src/cai_env/urdf/table.urdf.xacro (robot description, xacro)
@@ -44,5 +44,14 @@
     </collision>
     <gazebo reference="table">
-      <material>Gazebo/Green </material>
+      <!-- <material>Gazebo/Green </material> -->
+      <gravity>bool</gravity>
+      <maxVel>100</maxVel>
+      <kd>1</kd>
+      <maxContacts>20</maxContacts>
+      <mu2>1000000000000</mu2>
+      <selfCollide>10</selfCollide>
+      <mu1>1000000000000</mu1>
+      <minDepth>2</minDepth>
+      <kp>1000000000000.0</kp>
     </gazebo>
   </link>

Commit message: 修改了电池包的摩擦系数，暂时感觉良好

File: rokae/src/battery_pack_describe/urdf/v_battery.xacro (robot description, xacro)
@@ -3,6 +3,5 @@
      Commit Version: 1.5.1-0-g916b5db  Build Version: 1.5.7152.31018
      For more information, please see http://wiki.ros.org/sw_urdf_exporter -->
-<robot
-  name="v_battery">
+<robot  name="v_battery">
   <link    name="v_battery_base_link"  xmlns:xacro="http://www.ros.org/wiki/xacro">
     <inertial>
@@ -44,12 +43,21 @@
   </link>
   <gazebo reference="v_battery_base_link">
+    <!-- <material>Gazebo/GreyTransparent</material> -->
+    <kp>1000000.0</kp>
+    <kd>100.0</kd>
+    <mu1>50000000000000000000.0</mu1>
+    <mu2>50000000000000000000.0</mu2>
+    <maxVel>0</maxVel>
+    <minDepth>0.001</minDepth>
+  </gazebo>
+  <!-- <gazebo reference="v_battery_base_link">
       <maxVel>100</maxVel>
       <kd>200</kd>
       <maxContacts>200</maxContacts>
-      <mu2>5000000000000</mu2>
+      <mu2>50000000000000000000</mu2>
       <selfCollide>10</selfCollide>
-      <mu1>5000000000000</mu1>
+      <mu1>50000000000000000000</mu1>
       <minDepth>10</minDepth>
-      <kp>1000000000000.0</kp>
+      <kp>1000000000000.0</kp> -->
       <!-- <gravity>bool</gravity> -->
       <!-- <gravity>bool</gravity> -->
@@ -62,5 +70,5 @@
       <minDepth>10</minDepth>
       <kp>1</kp> -->
-  </gazebo>
+  <!-- </gazebo>  -->
   <link    name="v_battery_bolt_Link">
     <inertial>
@@ -104,5 +112,5 @@
 https://whtqh.gitbooks.io/gazebo_simu_chs/content/using_a_urdf_model.html  摩擦力和其他参数，定义链接
 -->
-  <gazebo reference="v_battery_bolt_Link">
+  <!-- <gazebo reference="v_battery_bolt_Link">
       <maxVel>0.01</maxVel>
       <kd>1</kd>
@@ -114,5 +122,5 @@
       <kp>1000000000000.0</kp>
     <material>Gazebo/Grey </material>
-</gazebo>
+</gazebo> -->
   <joint
     name="v_battery_bolt_joint"
@@ -168,5 +176,5 @@
     </collision>
   </link>
-  <gazebo reference="v_battery_nut_Link">
+  <!-- <gazebo reference="v_battery_nut_Link">
     <mu1>0.1</mu1>
     <mu2>0.1</mu2>
@@ -177,5 +185,5 @@
     <fdir1>1 0 0</fdir1>
     <material>Gazebo/FlatBlack</material>
-  </gazebo>
+  </gazebo> -->
   <joint
     name="v_battery_nut_joint"

Commit message: 电池包的修改

File: rokae/src/battery_pack_describe/urdf/v_battery.xacro (robot description, xacro)
@@ -112,15 +112,15 @@
 https://whtqh.gitbooks.io/gazebo_simu_chs/content/using_a_urdf_model.html  摩擦力和其他参数，定义链接
 -->
-  <!-- <gazebo reference="v_battery_bolt_Link">
+  <gazebo reference="v_battery_bolt_Link">
       <maxVel>0.01</maxVel>
       <kd>1</kd>
       <maxContacts>20</maxContacts>
-      <mu2>50000</mu2>
+      <mu2>5000000000000000</mu2>
       <selfCollide>0</selfCollide>
-      <mu1>50000</mu1>
+      <mu1>5000000000000000</mu1>
       <minDepth>0</minDepth>
       <kp>1000000000000.0</kp>
     <material>Gazebo/Grey </material>
-</gazebo> -->
+  </gazebo>
   <joint
     name="v_battery_bolt_joint"

File: rokae/src/rokae_desk/urdf/robot_tool_complex.xacro (robot description, xacro)
@@ -8,4 +8,5 @@
   <xacro:include filename="$(find realsense2_description)/urdf/gloal_d435_camera.urdf.xacro"   />
   <xacro:include filename="$(find battery_pack_describe)/urdf/weilan.urdf" />
+  <!-- <xacro:include filename="$(find battery_pack_describe)/urdf/v_battery.xacro"   /> -->
   <joint name="weilan_joint" type="fixed">
     <origin xyz="0 0 0.05" rpy="0 0 0" />
@@ -19,7 +20,7 @@
   </joint>
   <!-- <joint name="battery_pack_joint" type="fixed">
-    <origin xyz="0 0 0.12" rpy="0 0 3.14" />
+    <origin xyz="0 0 0.1000002" rpy="0 0 3.14" />
     <parent link="table"/>
-    <child link="battery_pack_link"/>
+    <child link="v_battery_base_link"/>
   </joint> -->
   <joint name="taotong_tool_joint" type="fixed">

Commit message: 电池不好加 碰撞盒

File: rokae/src/battery_pack_describe/urdf/v_battery.xacro (robot description, xacro)
@@ -28,5 +28,5 @@
       <origin     xyz="0 0 0"    rpy="0 0 0" />
       <geometry>
-        <box size="0.5 0.5 0.05" />
+        <!-- <box size="0.5 0.5 0.05" /> -->
         <mesh
           filename="package://battery_pack_describe/meshes/v_battery_base_link.dae" />
@@ -88,5 +88,5 @@
       <origin   xyz="0 0 0"   rpy="0 0 0" />
       <geometry>
-        <cylinder length="0.1" radius="0.02"/>
+        <cylinder length="0.002" radius="0.002"/>
         <mesh   filename="package://battery_pack_describe/meshes/v_battery_bolt_Link_metal.dae" />
       </geometry>
@@ -148,5 +148,5 @@
       <origin        xyz="0 0 0"        rpy="0 0 0" />
       <geometry>
-        <cylinder length="0.04" radius="0.02"/>
+        <!-- <cylinder length="0.001" radius="0.02"/> -->
         <mesh   filename="package://battery_pack_describe/meshes/v_battery_nut_Link.dae" />
       </geometry>

Commit message: 电池包的 碰撞调整

File: rokae/src/battery_pack_describe/urdf/v_battery.xacro (robot description, xacro)
@@ -3,32 +3,26 @@
      Commit Version: 1.5.1-0-g916b5db  Build Version: 1.5.7152.31018
      For more information, please see http://wiki.ros.org/sw_urdf_exporter -->
-<robot  name="v_battery">
-  <link    name="v_battery_base_link"  xmlns:xacro="http://www.ros.org/wiki/xacro">
+<robot name="v_battery">
+  <link name="v_battery_base_link"
+    xmlns:xacro="http://www.ros.org/wiki/xacro">
     <inertial>
-      <origin   xyz="-0.17823 0.0014541 -0.18254"  rpy="0 0 0" />
-      <mass        value="2.1452" />
-      <inertia
-        ixx="0.04437"
-        ixy="-0.00066651"
-        ixz="-0.0054047"
-        iyy="0.089539"
-        iyz="-0.0010719"
-        izz="0.045613" />
+      <origin xyz="-0.17823 0.0014541 -0.18254" rpy="0 0 0" />
+      <mass value="2.1452" />
+      <inertia ixx="0.04437" ixy="-0.00066651" ixz="-0.0054047" iyy="0.089539" iyz="-0.0010719" izz="0.045613" />
     </inertial>
     <visual>
-      <origin   xyz="0 0 0"   rpy="0 0 0" />
+      <origin xyz="0 0 0" rpy="0 0 0" />
       <geometry>
-        <mesh     filename="package://battery_pack_describe/meshes/v_battery_base_link.dae" />
+        <mesh filename="package://battery_pack_describe/meshes/v_battery_base_link.dae" />
       </geometry>
-      <material     name="">
-        <color    rgba="0.79216 0.81961 0.93333 1" />
+      <material name="">
+        <color rgba="0.79216 0.81961 0.93333 1" />
       </material>
     </visual>
     <collision>
-      <origin     xyz="0 0 0"    rpy="0 0 0" />
+      <origin xyz="0 0 0" rpy="0 0 0" />
       <geometry>
         <!-- <box size="0.5 0.5 0.05" /> -->
-        <mesh
-          filename="package://battery_pack_describe/meshes/v_battery_base_link.dae" />
+        <mesh filename="package://battery_pack_describe/meshes/v_battery_base_link.dae" />
       </geometry>
     </collision>
@@ -52,7 +46,7 @@
       <minDepth>10</minDepth>
       <kp>1000000000000.0</kp> -->
-      <!-- <gravity>bool</gravity> -->
-      <!-- <gravity>bool</gravity> -->
-      <!-- <maxVel>100</maxVel>
+  <!-- <gravity>bool</gravity> -->
+  <!-- <gravity>bool</gravity> -->
+  <!-- <maxVel>100</maxVel>
       <kd>10</kd>
       <maxContacts>200</maxContacts>
@@ -63,91 +57,67 @@
       <kp>1</kp> -->
   <!-- </gazebo>  -->
-  <link    name="v_battery_bolt_Link">
+  <link name="v_battery_bolt_Link">
     <inertial>
-      <origin     xyz="-0.00224797355412683 -2.42669320749123E-09 1.13997717515746E-09"
-        rpy="0 0 0" />
-      <mass  value="0.010043058879212" />
-      <inertia
-        ixx="8.16036465000949E-08"
-        ixy="-2.67875420699996E-13"
-        ixz="1.25078148224805E-13"
-        iyy="1.22914699774063E-06"
-        iyz="5.9822890763516E-14"
-        izz="1.22914675774153E-06" />
+      <origin xyz="-0.00224797355412683 -2.42669320749123E-09 1.13997717515746E-09" rpy="0 0 0" />
+      <mass value="0.010043058879212" />
+      <inertia ixx="8.16036465000949E-08" ixy="-2.67875420699996E-13" ixz="1.25078148224805E-13" iyy="1.22914699774063E-06" iyz="5.9822890763516E-14" izz="1.22914675774153E-06" />
     </inertial>
     <visual>
-      <origin   xyz="0 0 0"  rpy="0 0 0" />
+      <origin xyz="0 0 0" rpy="0 0 0" />
       <geometry>
-        <mesh   filename="package://battery_pack_describe/meshes/v_battery_bolt_Link_metal.dae" />
+        <mesh filename="package://battery_pack_describe/meshes/v_battery_bolt_Link_metal.dae" />
       </geometry>
-      <material  name="">
-        <color  rgba="0.776470588235294 0.756862745098039 0.737254901960784 1" />
+      <material name="">
+        <color rgba="0.776470588235294 0.756862745098039 0.737254901960784 1" />
       </material>
     </visual>
     <collision>
-      <origin   xyz="0 0 0"   rpy="0 0 0" />
+      <origin xyz="0 0 0" rpy="0 0 0" />
       <geometry>
-        <cylinder length="0.002" radius="0.002"/>
-        <mesh   filename="package://battery_pack_describe/meshes/v_battery_bolt_Link_metal.dae" />
+        <!-- <cylinder length="0.002" radius="0.002"/> -->
+        <mesh filename="package://battery_pack_describe/meshes/v_battery_bolt_Link_metal.dae" />
       </geometry>
     </collision>
   </link>
-<!--摩擦力参考链接，我修改了mu的大小。 https://boschresearch.github.io/pcg_gazebo_pkgs/tutorials/parsers/urdf/robots/
+  <!--摩擦力参考链接，我修改了mu的大小。 https://boschresearch.github.io/pcg_gazebo_pkgs/tutorials/parsers/urdf/robots/
 https://whtqh.gitbooks.io/gazebo_simu_chs/content/using_a_urdf_model.html  摩擦力和其他参数，定义链接
 -->
   <gazebo reference="v_battery_bolt_Link">
-      <maxVel>0.01</maxVel>
-      <kd>1</kd>
-      <maxContacts>20</maxContacts>
-      <mu2>5000000000000000</mu2>
-      <selfCollide>0</selfCollide>
-      <mu1>5000000000000000</mu1>
-      <minDepth>0</minDepth>
-      <kp>1000000000000.0</kp>
+    <maxVel>0.01</maxVel>
+    <kd>1</kd>
+    <maxContacts>20</maxContacts>
+    <mu2>5000000000000000</mu2>
+    <selfCollide>0</selfCollide>
+    <mu1>5000000000000000</mu1>
+    <minDepth>0</minDepth>
+    <kp>1000000000000.0</kp>
     <material>Gazebo/Grey </material>
   </gazebo>
-  <joint
-    name="v_battery_bolt_joint"
-    type="continuous">
-    <origin
-      xyz="0.057323 -0.038452 0"
-      rpy="0.39309 1.5708 0" />
-    <parent
-      link="v_battery_base_link" />
-    <child
-      link="v_battery_bolt_Link" />
-    <axis
-      xyz="1 0 0" />
+  <joint name="v_battery_bolt_joint" type="continuous">
+    <origin xyz="0.057323 -0.038452 0" rpy="0.39309 1.5708 0" />
+    <parent link="v_battery_base_link" />
+    <child link="v_battery_bolt_Link" />
+    <axis xyz="1 0 0" />
   </joint>
-  <link
-    name="v_battery_nut_Link">
+  <link name="v_battery_nut_Link">
     <inertial>
-      <origin
-        xyz="-8.23260362659006E-10 1.38777878078145E-17 -0.0026006024331304"
-        rpy="0 0 0" />
-      <mass
-        value="0.00265736664598247" />
-      <inertia
-        ixx="2.79753045005072E-08"
-        ixy="5.04580173657347E-23"
-        ixz="1.31793951411467E-18"
-        iyy="2.79771327058771E-08"
-        iyz="-4.83267733699208E-14"
-        izz="4.46160415460721E-08" />
+      <origin xyz="-8.23260362659006E-10 1.38777878078145E-17 -0.0026006024331304" rpy="0 0 0" />
+      <mass value="0.00265736664598247" />
+      <inertia ixx="2.79753045005072E-08" ixy="5.04580173657347E-23" ixz="1.31793951411467E-18" iyy="2.79771327058771E-08" iyz="-4.83267733699208E-14" izz="4.46160415460721E-08" />
     </inertial>
     <visual>
-      <origin   xyz="0 0 0"  rpy="0 0 0" />
+      <origin xyz="0 0 0" rpy="0 0 0" />
       <geometry>
-        <mesh    filename="package://battery_pack_describe/meshes/v_battery_nut_Link.dae" />
+        <mesh filename="package://battery_pack_describe/meshes/v_battery_nut_Link.dae" />
       </geometry>
-      <material     name="">
-        <color    rgba="0.776470588235294 0.756862745098039 0.737254901960784 1" />
+      <material name="">
+        <color rgba="0.776470588235294 0.756862745098039 0.737254901960784 1" />
       </material>
     </visual>
     <collision>
-      <origin        xyz="0 0 0"        rpy="0 0 0" />
+      <origin xyz="0 0 0" rpy="0 0 0" />
       <geometry>
         <!-- <cylinder length="0.001" radius="0.02"/> -->
-        <mesh   filename="package://battery_pack_describe/meshes/v_battery_nut_Link.dae" />
+        <mesh filename="package://battery_pack_describe/meshes/v_battery_nut_Link.dae" />
       </geometry>
     </collision>
@@ -163,16 +133,9 @@
     <material>Gazebo/FlatBlack</material>
   </gazebo> -->
-  <joint
-    name="v_battery_nut_joint"
-    type="fixed">
-    <origin
-      xyz="0.057323 -0.038452 0"
-      rpy="0 0 2.7485" />
-    <parent
-      link="v_battery_base_link" />
-    <child
-      link="v_battery_nut_Link" />
-    <axis
-      xyz="0 0 -1" />
+  <joint name="v_battery_nut_joint" type="fixed">
+    <origin xyz="0.057323 -0.038452 0" rpy="0 0 2.7485" />
+    <parent link="v_battery_base_link" />
+    <child link="v_battery_nut_Link" />
+    <axis xyz="0 0 -1" />
   </joint>
 </robot>
