Commit message: ur rviz

File: rokae/src/universal_robot/ur_e_description/urdf/ur10e_joint_limited_robot.urdf.xacro (robot description, xacro)
@@ -1,5 +1,4 @@
 <?xml version="1.0"?>
-<robot xmlns:xacro="http://ros.org/wiki/xacro"
-       name="ur10e" >
+<robot xmlns:xacro="http://ros.org/wiki/xacro" name="ur10e">
   <!-- common stuff -->
   <xacro:include filename="$(find ur_e_description)/urdf/common.gazebo.xacro" />
@@ -7,17 +6,40 @@
   <xacro:include filename="$(find ur_e_description)/urdf/ur10e.urdf.xacro" />
   <!-- arm -->
-  <xacro:ur10e_robot prefix="" joint_limited="true"
-		 shoulder_pan_lower_limit="${-pi}" shoulder_pan_upper_limit="${pi}"
-		 shoulder_lift_lower_limit="${-pi}" shoulder_lift_upper_limit="${pi}"
-		 elbow_joint_lower_limit="${-pi}" elbow_joint_upper_limit="${pi}"
-		 wrist_1_lower_limit="${-pi}" wrist_1_upper_limit="${pi}"
-		 wrist_2_lower_limit="${-pi}" wrist_2_upper_limit="${pi}"
-		 wrist_3_lower_limit="${-pi}" wrist_3_upper_limit="${pi}"
-/>
+  <xacro:ur10e_robot prefix="" joint_limited="true" shoulder_pan_lower_limit="${-pi}" shoulder_pan_upper_limit="${pi}" shoulder_lift_lower_limit="${-pi}" shoulder_lift_upper_limit="${pi}" elbow_joint_lower_limit="${-pi}" elbow_joint_upper_limit="${pi}" wrist_1_lower_limit="${-pi}" wrist_1_upper_limit="${pi}" wrist_2_lower_limit="${-pi}" wrist_2_upper_limit="${pi}" wrist_3_lower_limit="${-pi}" wrist_3_upper_limit="${pi}" />
+  <xacro:include filename="$(find cai_env)/urdf/ur_table.urdf.xacro" />
+  <xacro:include filename="$(find battery_pack_describe)/urdf/weilan.urdf" />
+  <xacro:include filename="$(find rokae_desk)/urdf/camera_taotong.xacro" />
+  <xacro:include filename="$(find realsense2_description)/urdf/test_d435_camera_ur.urdf.xacro" />
+  <xacro:include filename="$(find realsense2_description)/urdf/gloal_d435_camera.urdf.xacro" />
   <link name="world" />
+  <joint name="table_joint" type="fixed">
+    <origin xyz="0.0 0.0 0.0" rpy="0.0 0.0 0.0" />
+    <parent link="world"/>
+    <child link="world_table"/>
+  </joint>
   <joint name="world_joint" type="fixed">
-    <parent link="world" />
+    <parent link="world_table" />
     <child link = "base_link" />
-    <origin xyz="0.0 0.0 0.0" rpy="0.0 0.0 0.0" />
+    <origin xyz="-0.55 0 0.92" rpy="0 0 0" />
+  </joint>
+  <joint name="weilan_joint" type="fixed">
+    <origin xyz="0 0 0.85" rpy="0 0 0" />
+    <parent link="world_table"/>
+    <child link="weilan"/>
+  </joint>
+  <joint name="taotong_tool_joint" type="fixed">
+    <origin xyz="0 0 0" rpy="0 3.14 0" />
+    <parent link="tool0"/>
+    <child link="tool_base_link"/>
+  </joint>
+  <joint name="arm_camera_joint" type="fixed">
+    <origin xyz="0 -0.02 0.10" rpy="0 -1.57 1.57"/>
+    <parent link="tool0"/>
+    <child link="world_base"/>
+  </joint>
+  <joint name="scene_camera_joint" type="fixed">
+    <origin xyz="0 0 2.30" rpy="0 1.57 1.57"/>
+    <parent link="world"/>
+    <child link="gloal_world_base"/>
   </joint>
 </robot>

File: rokae/src/universal_robot/ur_e_description/urdf/ur10e_robot.urdf.xacro (robot description, xacro)
@@ -1,5 +1,4 @@
 <?xml version="1.0"?>
-<robot xmlns:xacro="http://ros.org/wiki/xacro"
-       name="ur10e" >
+<robot xmlns:xacro="http://ros.org/wiki/xacro" name="ur10e">
   <!-- common stuff -->
   <xacro:include filename="$(find ur_e_description)/urdf/common.gazebo.xacro" />
@@ -8,9 +7,39 @@
   <!-- arm -->
   <xacro:ur10e_robot prefix="" joint_limited="false"/>
+  <xacro:include filename="$(find cai_env)/urdf/ur_table.urdf.xacro" />
+  <xacro:include filename="$(find battery_pack_describe)/urdf/weilan.urdf" />
+  <xacro:include filename="$(find rokae_desk)/urdf/camera_taotong.xacro" />
+  <xacro:include filename="$(find realsense2_description)/urdf/test_d435_camera_ur.urdf.xacro" />
+  <xacro:include filename="$(find realsense2_description)/urdf/gloal_d435_camera.urdf.xacro" />
   <link name="world" />
+  <joint name="table_joint" type="fixed">
+    <origin xyz="0.0 0.0 0.0" rpy="0.0 0.0 0.0" />
+    <parent link="world"/>
+    <child link="world_table"/>
+  </joint>
   <joint name="world_joint" type="fixed">
-    <parent link="world" />
+    <parent link="world_table" />
     <child link = "base_link" />
-    <origin xyz="0.0 0.0 0.0" rpy="0.0 0.0 0.0" />
+    <origin xyz="-0.55 0 0.92" rpy="0 0 0" />
+  </joint>
+  <joint name="weilan_joint" type="fixed">
+    <origin xyz="0 0 0.85" rpy="0 0 0" />
+    <parent link="world_table"/>
+    <child link="weilan"/>
+  </joint>
+  <joint name="taotong_tool_joint" type="fixed">
+    <origin xyz="0 0 0" rpy="0 3.14 0" />
+    <parent link="tool0"/>
+    <child link="tool_base_link"/>
+  </joint>
+  <joint name="arm_camera_joint" type="fixed">
+    <origin xyz="0 -0.02 0.10" rpy="0 -1.57 1.57"/>
+    <parent link="tool0"/>
+    <child link="world_base"/>
+  </joint>
+  <joint name="scene_camera_joint" type="fixed">
+    <origin xyz="0 0 2.30" rpy="0 1.57 1.57"/>
+    <parent link="world"/>
+    <child link="gloal_world_base"/>
   </joint>
 </robot>
